File: ADC3_FPGA_BGA.brd (EAGLE design)
At the start: 84.8 x 100.8 mm, 129 parts, among them CON1 2X17-FEMALE, IC1 3.3V, IC2 1.8V, IC3 1.0V, IC4 LFD2NX-40, IC5 EEPROM, IC6 AE-FT232HL, J1 SJ-1608, J2 SJ-1608, J3 IO0, J4 IO2, J5 IO6, J6 IO3, J7 IO4, SW1 5V, U1 DC-DC, X1 OSC

Commit message: 発注
Parts:
- added FB3: FB, my_rcl:1608-J
- added J8: 1.0V, my_rcl:1608-J
- added TP23: TX, my_connector:TESTPIN
- added TP24: GND, my_connector:TESTPIN
- moved DR3 8.16 mm to (30.4, -70.4)
- moved DR4 8.00 mm to (30.4, 22.4)
- moved DR1 1.60 mm to (-40.0, -70.4)
- moved C25 0.20 mm to (-5.00, -0.20)
- turned C1 to 180 degrees
Connections:
- net CLK_25M renamed CLK_20M
- new net +1V0CORE: C12.1, C14.1, C17.1, C9.1, IC4.F9, IC4.G7, IC4.H9, IC4.J7, IC4.J9, J8.2, TP3.1
- new net N$9: FB3.2, SW1.2
- new net UART_TX: IC4.C4, TP23.1
- net +1V0: now also J8.1; no longer C12.1, C14.1, C17.1, C9.1, IC4.F9, IC4.G7, IC4.H9, IC4.J7, IC4.J9, TP3.1
- net +5V: now also FB3.1; no longer SW1.2
- net GND: now also TP24.1
Routing:
- net +1V0: track 52.4 -> 6.20 mm, vias 6 -> 0
- net +1V0CORE: track 0.00 -> 44.8 mm, vias 0 -> 6
- net UART_TX: track 0.00 -> 14.1 mm, vias 0 -> 1
- net N$9: track 0.00 -> 6.05 mm
- net VCCIO4: track 75.9 -> 72.7 mm
- net +1V8: track 150.4 -> 153.4 mm
- net VCCIO3: track 44.7 -> 47.1 mm
- net FLASH_CS: track 32.1 -> 29.9 mm
- net LV_IO28: track 24.6 -> 26.1 mm
- net +5V: track 11.2 -> 12.2 mm
- net FT_CLK: track 22.2 -> 22.7 mm
Other:
- board size 84.8 x 100.8 mm -> 77.6 x 100 mm
- board text added: "NX FPGA Board ver1"

Commit message: メザニンコネクタ
Parts:
- removed C1, C17, C18, C19, C20, C21, C22, C23, C5: 10u, my_rcl:3225
- removed C2, C9: 0.1u, my_rcl:1608
- removed D4: LED3, my_rcl:D1608
- removed DR1, DR2, DR3, DR4: HOLE-3.2, my_connector:HOLE_3.2
- removed F1: 0.9A, my_rcl:3216
- removed FB3: FB, my_rcl:1608-J
- removed IC1: 3.3V, my_ic:TO220-SOP-DUAL
- removed J3: IO0, my_rcl:1608-J
- removed J4: IO2, my_rcl:1608-J
- removed J5: IO6, my_rcl:1608-J
- removed J6: IO3, my_rcl:1608-J
- removed J7: IO4, my_rcl:1608-J
- removed J8: 1.0V, my_rcl:1608-J
- removed JP1: JTAG, my_connector:1X07
- removed JP2: SPI, my_connector:1X07
- removed JP3: LVIO, pinhead:2X20
- removed JP4: HVIO, pinhead:2X03
- removed R1: 22, my_rcl:1608-J
- removed R18, R26: D1, my_rcl:1608-J
- removed R20, R30: D5, my_rcl:1608-J
- removed R21, R32: D7, my_rcl:1608-J
- removed R22: D9, my_rcl:1608-J
- removed R23: D11, my_rcl:1608-J
- removed R24: D13, my_rcl:1608-J
- removed R25: D0, my_rcl:1608-J
- removed R27: D2, my_rcl:1608-J
- removed R28: D3, my_rcl:1608-J
- removed R29: D4, my_rcl:1608-J
- removed R31: D6, my_rcl:1608-J
- removed R33: CLK, my_rcl:1608-J
- removed R34: WR, my_rcl:1608-J
- removed R35: RD, my_rcl:1608-J
- removed R36: TXNE, my_rcl:1608-J
- removed R37: RXNF, my_rcl:1608-J
- removed R38, R39, R40, R41, R42: 1k, my_rcl:1608
- removed SW1: 5V, my_connector:1X03
- removed TP1: ADCP, my_connector:TESTPAD
- removed TP10, TP22, TP24: GND, my_connector:TESTPIN
- removed TP11, TP12, TP13, TP14, TP15, TP16, TP17, TP18: (no value), my_connector:TESTPAD
- removed TP19: VIN+, my_connector:TESTPIN
- removed TP2: ADCN, my_connector:TESTPAD
- removed TP20: VIN-, my_connector:TESTPIN
- removed TP21: FT_+5V, my_connector:TESTPIN
- removed TP23: TX, my_connector:TESTPIN
- removed TP3: 1.0V, my_connector:TESTPIN
- removed TP4: 1.8V, my_connector:TESTPIN
- removed TP5: VCCIO0, my_connector:TESTPIN
- removed TP6: VCCIO2, my_connector:TESTPIN
- removed TP7: VCCIO6, my_connector:TESTPIN
- removed TP8: VCCIO3, my_connector:TESTPIN
- removed TP9: VCCIO4, my_connector:TESTPIN
- removed U1: DC-DC, my_ic:DCDC
- removed X1: OSC, my_rcl:KC3225
- added C33, C36: 10u, my_rcl:1608
- added C34, C35: 0.1u, my_rcl:1608
- added CON2, CON3: MEZZANINE_2X30, my_connector:MEZZANINE_0.8MM_2X30
- added IC7: FT2232H, my_ic:VQFN56
- added IC8: HYPERRAM, my_ic:TFBGA24
- added X2: 12MHz, my_rcl:KC3225
- C10, C12, C13, C14, C15, C16, C24, C25: device my_rcl:1608 -> my_rcl:1005
- C30: value 0.1u -> 10u
- C31, C32: value 100u -> 22p; device my_rcl:E2,5-8 -> my_rcl:1608
- CON1: value 2X17-FEMALE -> USB-A; device my_connector:2X17/90 -> my_connector:UX60A-MB-5ST
- IC6: value AE-FT232HL -> 93LC56; device my_ic:AE-FT232HL -> my_ic:SOT23-6
- R11: value D0 -> 10k; device my_rcl:1608-J -> my_rcl:1608
- R12: value D2 -> 1k; device my_rcl:1608-J -> my_rcl:1608
- R13: value D4 -> 12.1k; device my_rcl:1608-J -> my_rcl:1608
- R14: value D6 -> 1k; device my_rcl:1608-J -> my_rcl:1608
- R15: value D8 -> 1k; device my_rcl:1608-J -> my_rcl:1608
- R16: value D10 -> 1k; device my_rcl:1608-J -> my_rcl:1608
- R17: value D12 -> 1k; device my_rcl:1608-J -> my_rcl:1608
- R19: value D3 -> 1k; device my_rcl:1608-J -> my_rcl:1608
- moved FB2 91.4 mm to (-26.8, 20.0), turned to 270 degrees
- moved C4 80.6 mm to (-47.2, 32.8)
- moved C3 75.8 mm to (-43.2, 32.8)
- moved C8 73.0 mm to (-54.4, 32.8), flipped to the top
- moved J1 69.6 mm to (-1.40, 29.2), turned to 90 degrees
- moved J2 69.2 mm to (3.00, 29.2), turned to 90 degrees
- moved C28 65.9 mm to (-53.6, 39.2), flipped to the top, turned to 0 degrees
- moved C11 64.6 mm to (-51.2, 32.8), flipped to the top, turned to 0 degrees
- moved D5 64.0 mm to (-33.4, -1.60)
- moved FB1 63.4 mm to (-24.4, -10.2)
- moved C32 62.6 mm to (-9.60, -8.20), turned to 180 degrees
- moved C27 60.8 mm to (-49.6, 39.2), flipped to the top
- moved R19 54.5 mm to (-33.4, -5.20), turned to 90 degrees
- moved C26 54.1 mm to (-45.6, 39.2), flipped to the top
- moved R17 54.0 mm to (-31.8, -5.20), turned to 90 degrees
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Connections:
- removed net +1V0CORE: C12.1, C14.1, C17.1, C9.1, IC4.F9, IC4.G7, IC4.H9, IC4.J7, IC4.J9, J8.2, TP3.1
- removed net +5V: C1.1, C2.1, FB3.1, IC1.1, IC1.4
- removed net +5VD: SW1.1, U1.+5VD
- removed net ADC_D0: IC4.E1, R11.2
- removed net ADC_D1: IC4.E2, R18.1
- removed net ADC_D10: IC4.F3, R16.2
- removed net ADC_D11: IC4.F4, R23.1
- removed net ADC_D12: IC4.H3, R17.2
- removed net ADC_D13: IC4.H4, R24.1
- removed net ADC_D2: IC4.F1, R12.2
- removed net ADC_D3: IC4.F2, R19.1
- removed net ADC_D4: IC4.G1, R13.2
- removed net ADC_D5: IC4.G2, R20.1
- removed net ADC_D6: IC4.H1, R14.2
- removed net ADC_D7: IC4.H2, R21.1
- removed net ADC_D8: IC4.J1, R15.2
- removed net ADC_D9: IC4.J2, R22.1
- removed net CLK_20M: IC4.B12, R1.2
- removed net FT_+5V: F1.2, SW1.3, TP21.1
- removed net FT_RD: IC4.E12, R35.2
- removed net FT_WR: IC4.G14, R34.2
- removed net HV_IO0: IC4.C3, JP4.3
- removed net HV_IO1: IC4.B1, JP4.4
- removed net HV_IO2: IC4.C2, JP4.5
- removed net HV_IO3: IC4.C1, JP4.6
- removed net LED3: D4.A, IC4.A12
- removed net LV_IO0: IC4.K1, JP3.3
- removed net LV_IO1: IC4.K3, JP3.4
- removed net LV_IO10: IC4.N4, JP3.13
- removed net LV_IO11: IC4.P4, JP3.14
- removed net LV_IO12: IC4.N5, JP3.15
- removed net LV_IO13: IC4.P5, JP3.16
- removed net LV_IO14: IC4.N6, JP3.17
- removed net LV_IO15: IC4.P6, JP3.18
- removed net LV_IO16: IC4.M8, JP3.23
- removed net LV_IO17: IC4.P8, JP3.24
- removed net LV_IO18: IC4.N8, JP3.25
- removed net LV_IO19: IC4.P9, JP3.26
- removed net LV_IO2: IC4.L1, JP3.5
- removed net LV_IO20: IC4.N9, JP3.27
- removed net LV_IO21: IC4.P10, JP3.28
- removed net LV_IO22: IC4.N10, JP3.29
- removed net LV_IO23: IC4.P11, JP3.30
- removed net LV_IO24: IC4.N11, JP3.31
- removed net LV_IO25: IC4.P12, JP3.32
- removed net LV_IO26: IC4.L13, JP3.33
- removed net LV_IO27: IC4.P13, JP3.34
- removed net LV_IO28: IC4.N13, JP3.35
- removed net LV_IO29: IC4.N14, JP3.36
- removed net LV_IO3: IC4.L2, JP3.6
- removed net LV_IO30: IC4.M13, JP3.37
- removed net LV_IO31: IC4.M14, JP3.38
- removed net LV_IO4: IC4.M1, JP3.7
- removed net LV_IO5: IC4.M2, JP3.8
- removed net LV_IO6: IC4.N1, JP3.9
- removed net LV_IO7: IC4.P2, JP3.10
- removed net LV_IO8: IC4.L3, JP3.11
- removed net LV_IO9: IC4.P3, JP3.12
- removed net N$17: IC6.10, R28.2
- removed net N$18: IC6.11, R29.2
- removed net N$19: IC6.12, R30.2
- removed net N$20: FB1.1, U1.V+
- removed net N$21: FB2.2, U1.V-
- removed net N$5: D4.K, R41.2
- removed net N$6: TP20.1, U1.VIN-
- removed net N$61: CON1.31, R17.1
- removed net N$62: CON1.27, R16.1
- removed net N$63: CON1.23, R15.1
- removed net N$64: CON1.19, R14.1
- removed net N$65: CON1.15, R13.1
- removed net N$66: CON1.11, R12.1
- removed net N$67: CON1.7, R11.1
- removed net N$68: CON1.10, R18.2
- removed net N$69: CON1.14, R19.2
- removed net N$7: TP19.1, U1.VIN+
- removed net N$70: CON1.18, R20.2
- removed net N$71: CON1.22, R21.2
- removed net N$72: CON1.26, R22.2
- removed net N$73: CON1.30, R23.2
- removed net N$74: CON1.34, R24.2
- removed net N$75: IC6.13, R31.2
- removed net N$76: IC6.14, R32.2
- removed net N$77: IC6.17, R35.1
- removed net N$78: F1.1, IC6.27
- removed net N$8: R1.1, X1.3
- removed net UART_TX: IC4.C4, TP23.1
- removed net V+: C31.+, CON1.3, CON1.4, FB1.2
- removed net V-: C32.-, CON1.1, CON1.2, FB2.1
- removed net VCCIO2: C20.1, C25.1, IC4.G11, J4.2, TP6.1
- removed net VCCIO3: C22.1, C26.1, IC4.M10, IC4.N12, J6.2, TP8.1
- removed net VCCIO4: C23.1, C28.1, IC4.L5, IC4.N3, J7.2, JP3.19, JP3.22, TP9.1
- removed net VCCIO6: C21.1, C29.1, C30.1, IC4.E4, IC4.G4, J5.2, TP7.1
- new net DRAM_+1V8: C36.1, FB2.1, IC8.B4, IC8.D1, IC8.E4
- new net DRAM_CKN: IC4.L7, IC8.B1
- new net DRAM_CKP: IC4.M7, IC8.B2
- new net DRAM_CS: IC4.K6, IC8.A3
- new net DRAM_DQ0: IC4.N5, IC8.D3
- new net DRAM_DQ1: IC4.P7, IC8.D2
- new net DRAM_DQ2: IC4.P4, IC8.C4
- new net DRAM_DQ3: IC4.N4, IC8.D4
- new net DRAM_DQ4: IC4.M4, IC8.D5
- new net DRAM_DQ5: IC4.P5, IC8.E3
- new net DRAM_DQ6: IC4.P6, IC8.E2
- new net DRAM_DQ7: IC4.N6, IC8.E1
- new net DRAM_NRST: IC4.K5, IC8.A4
- new net DRAM_RWDS: IC4.N7, IC8.C3
- new net FT_+1V8: C33.1, IC7.2, IC7.31, IC7.43
- new net FT_+3V3: C30.1, FB1.2, IC6.6, IC7.16, IC7.36, IC7.44, IC7.5, IC7.50, IC7.9, R11.1, R14.1
- new net FT_NOE: IC4.D6, IC7.28
- new net FT_NRD: IC4.C5, IC7.24
- new net FT_NWR: IC4.C6, IC7.25
- new net FT_SIWU: IC4.D5, IC7.26
- new net IOH0: CON2.50, IC4.C14
- new net IOH1: CON2.48, IC4.D12
- new net IOH10: CON2.39, IC4.E12
- new net IOH100: CON3.18, IC4.J4
- new net IOH101: CON3.20, IC4.J3
- new net IOH102: CON3.22, IC4.H4
- new net IOH103: CON3.24, IC4.H3
- new net IOH104: CON3.26, IC4.F4
- new net IOH105: CON3.28, IC4.F3
- new net IOH106: CON3.17, IC4.J2
- new net IOH107: CON3.19, IC4.J1
- new net IOH108: CON3.21, IC4.H2
- new net IOH109: CON3.23, IC4.H1
- new net IOH11: CON2.37, IC4.E11
- new net IOH110: CON3.25, IC4.G2
- new net IOH111: CON3.27, IC4.G1
- new net IOH112: CON3.29, IC4.F2
- new net IOH113: CON3.31, IC4.F1
- new net IOH114: CON3.30, IC4.E2
- new net IOH115: CON3.32, IC4.E1
- new net IOH12: CON2.35, IC4.F11
- new net IOH13: CON2.33, IC4.G12
- new net IOH14: CON2.47, IC4.C11
- new net IOH15: CON2.51, IC4.A12
- new net IOH16: CON2.49, IC4.A10
- new net IOH17: CON2.40, IC4.F13
- new net IOH18: CON2.42, IC4.E14
- new net IOH2: CON2.46, IC4.D14
- new net IOH3: CON2.44, IC4.E13
- new net IOH4: CON2.38, IC4.F14
- new net IOH5: CON2.36, IC4.G13
- new net IOH6: CON2.34, IC4.G14
- new net IOH7: CON2.45, IC4.E9
- new net IOH8: CON2.43, IC4.D11
- new net IOH9: CON2.41, IC4.E10
- new net IOL0: CON2.26, IC4.J14
- new net IOL1: CON2.24, IC4.J13
- new net IOL10: CON2.6, IC4.P13
- new net IOL101: CON3.4, IC4.P3
- new net IOL102: CON3.6, IC4.P2
- new net IOL103: CON3.8, IC4.N1
- new net IOL104: CON3.3, IC4.M2
- new net IOL105: CON3.5, IC4.M1
- new net IOL106: CON3.7, IC4.L2
- new net IOL107: CON3.9, IC4.L1
- new net IOL108: CON3.10, IC4.L3
- new net IOL109: CON3.12, IC4.K3
- new net IOL11: CON2.29, IC4.K9
- new net IOL110: CON3.11, IC4.K2
- new net IOL111: CON3.13, IC4.K1
- new net IOL12: CON2.27, IC4.K10
- new net IOL13: CON2.25, IC4.K11
- new net IOL14: CON2.23, IC4.K12
- new net IOL15: CON2.21, IC4.L9
- new net IOL16: CON2.19, IC4.L12
- new net IOL17: CON2.17, IC4.M9
- new net IOL18: CON2.15, IC4.M11
- new net IOL19: CON2.13, IC4.N11
- new net IOL2: CON2.22, IC4.K14
- new net IOL20: CON2.4, IC4.P12
- new net IOL21: CON2.11, IC4.P11
- new net IOL22: CON2.9, IC4.N10
- new net IOL23: CON2.7, IC4.P10
- new net IOL24: CON2.5, IC4.N9
- new net IOL25: CON2.3, IC4.P9
- new net IOL3: CON2.20, IC4.K13
- new net IOL4: CON2.18, IC4.L14
- new net IOL5: CON2.16, IC4.L13
- new net IOL6: CON2.14, IC4.M14
- new net IOL7: CON2.12, IC4.M13
- new net IOL8: CON2.10, IC4.N14
- new net IOL9: CON2.8, IC4.N13
- new net USB_+5V: CON1.1
- new net USB_DM: CON1.2, IC7.7
- new net USB_DP: CON1.3, IC7.8
- net +1V0: now also C12.1, C14.1, C8.1, IC4.F9, IC4.G7, IC4.H9, IC4.J7, IC4.J9; no longer J8.1
- net +1V8: now also C10.1, C26.1, C28.1, C29.1, FB2.2, IC4.L5, IC4.M10, IC4.N12, IC4.N3; no longer C11.1, C18.1, J6.1, J7.1, JP3.2, JP3.39, TP4.1
- net +3V3: now also C11.1, C24.1, C25.1, C34.1, C35.1, FB1.1, IC4.C12, IC4.C7, IC4.E4, IC4.G11, IC4.G4, R10.2, R2.2, R3.2, R5.2, R6.2, R7.2, R8.2, R9.2; no longer C5.1, IC1.3, IC1.6, J3.1, J4.1, J5.1, JP4.2
- net ADC_DN1: now also CON2.30; no longer TP2.1
- net ADC_DP1: now also CON2.28; no longer TP1.1
- net DONE: no longer JP2.6
- net FLASH_CS: no longer JP2.1
- net FLASH_MISO: no longer JP2.2
- net FLASH_MOSI: no longer JP2.5
- net FLASH_SCK: no longer JP2.3
- net FT_CLK: now also IC4.D7, IC7.27; no longer IC4.D11, R33.2
- net FT_D0: now also IC4.E3, IC7.12; no longer IC4.C14, R25.1
- net FT_D1: now also IC4.D2, IC7.13; no longer IC4.D12, R26.1
- net FT_D2: now also IC4.D1, IC7.14; no longer IC4.D14, R27.1
- net FT_D3: now also IC4.D3, IC7.15; no longer IC4.E13, R28.1
- net FT_D4: now also IC4.C1, IC7.17; no longer IC4.E14, R29.1
- net FT_D5: now also IC4.C2, IC7.18; no longer IC4.F13, R30.1
- net FT_D6: now also IC4.B1, IC7.19; no longer IC4.F14, R31.1
- net FT_D7: now also IC4.C3, IC7.20; no longer IC4.G13, R32.1
- net FT_RXNF: now also IC4.C4, IC7.22; no longer IC4.E11, R37.2
- net FT_TXNE: now also IC4.B5, IC7.23; no longer IC4.G12, R36.2
- net GND: now also C31.2, C32.2, C33.2, C34.2, C35.2, C36.2, CON1.M1, CON1.M2, CON1.M3, CON1.M4, CON2.1, CON2.2, CON2.31, CON2.32, CON3.1, CON3.14, CON3.15, CON3.16, CON3.2, IC6.2, IC7.10, IC7.21, IC7.41, IC7.45, IC7.HT, IC8.B3, IC8.C1, IC8.E5, R13.2, R15.1, R16.1, R17.1, R19.1, X2.2, X2.4; no longer C1.2, C17.2, C18.2, C19.2, C2.2, C20.2, C21.2, C22.2, C23.2, C31.-, C32.+, C5.2, C9.2, CON1.12, CON1.13, CON1.16, CON1.17, CON1.20, CON1.21, CON1.24, CON1.25, CON1.28, CON1.29, CON1.32, CON1.33, CON1.6, CON1.8, CON1.9, IC1.2, IC1.5, IC6.28, IC6.6, JP1.4, JP2.4, JP3.1, JP3.20, JP3.21, JP3.40, JP4.1, R38.1, R39.1, R40.1, R41.1, R42.1, TP10.1, TP11.1, TP12.1, TP13.1, TP14.1, TP15.1, TP16.1, TP17.1, TP18.1, TP22.1, TP24.1, U1.GND1, U1.GND2, X1.2
- net JTAG_EN: no longer JP1.6
- net JTAG_TCK: now also IC7.32; no longer JP1.3
- net JTAG_TDI: now also IC7.33; no longer JP1.2
- net JTAG_TDO: now also IC7.34; no longer JP1.5
- net JTAG_TMS: now also IC7.35; no longer JP1.1
- net LED0: now also IC4.B13; no longer IC4.B14
- net LED1: now also IC4.B14; no longer IC4.B13
- net LED2: now also IC4.B12; no longer IC4.C13
- net N$1: now also R19.2; no longer R42.2
- net N$10: now also IC6.3, IC7.55; no longer IC6.15, R37.1
- net N$11: now also IC6.5, IC7.1, R12.2; no longer IC6.16, R36.1
- net N$12: now also IC6.1, R11.2, R12.1; no longer IC6.18, R34.1
- net N$13: now also C32.1, IC7.4, X2.3; no longer IC6.20, R33.1
- net N$14: now also C31.1, IC7.3, X2.1; no longer IC6.7, R25.2
- net N$15: now also IC7.6, R13.1; no longer IC6.8, R26.2
- net N$16: now also IC7.11, R14.2; no longer IC6.9, R27.2
- net N$2: now also R15.2; no longer R38.2
- net N$3: now also R16.2; no longer R39.2
- net N$4: now also R17.2; no longer R40.2
- net N$9: now also IC6.4, IC7.56; no longer FB3.2, SW1.2
- net PROGRAMN: no longer JP2.7
- net VCCIO0: no longer C10.1, C19.1, C24.1, C8.1, IC4.C12, IC4.C7, J3.2, JP1.7, R10.2, R2.2, R3.2, R5.2, R6.2, R7.2, R8.2, R9.2, TP5.1, X1.1, X1.4
Routing:
- net VCCIO0: track 96.6 -> 0.00 mm, vias 5 -> 0
- net +1V8: track 153.4 -> 64.9 mm, vias 10 -> 15
- net VCCIO4: track 72.7 -> 0.00 mm, vias 2 -> 0
- net N$78: track 57.4 -> 0.00 mm
- net VCCIO3: track 47.1 -> 0.00 mm, vias 2 -> 0
- net V-: track 47.0 -> 0.00 mm
- net +1V0CORE: track 44.8 -> 0.00 mm, vias 6 -> 0
- net VCCIO6: track 44.3 -> 0.00 mm, vias 2 -> 0
- net V+: track 43.1 -> 0.00 mm
- net +3V3: track 71.7 -> 32.2 mm, vias 0 -> 5
- net FT_+3V3: track 0.00 -> 39.5 mm, vias 0 -> 7
- net VCCIO2: track 37.2 -> 0.00 mm, vias 1 -> 0
- net JTAG_EN: track 39.7 -> 4.14 mm, vias 1 -> 0
- net +1V0: track 6.20 -> 40.7 mm, vias 0 -> 8
- net HV_IO0: track 31.5 -> 0.00 mm
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- removed copper zone on layer 1, net GND
- removed copper zone on layer 15, net GND
- removed copper zone on layer 16, net GND
Other:
- board outline removed
- board text removed: "NX FPGA Board ver1"

Commit message: 4層DRC
Parts:
- removed C31, C32: 22p, my_rcl:1608
- removed C33, C36: 10u, my_rcl:1608
- removed C34, C35: 0.1u, my_rcl:1608
- removed J1, J2: SJ-1608, my_rcl:1608-J
- added C1, C18, C21, C22, C23, C5: 0.1u, my_rcl:1608
- added C17, C19, C9: 0.1u, my_rcl:1005
- added C2, C20: 10u, my_rcl:1608
- added D4: LED2, my_rcl:D1608
- added FB3: 1.8V, my_rcl:1608-J
- added FB4, FB6: FT, my_rcl:1608-J
- added FB5: DRAM, my_rcl:1608-J
- added IC1: 3.3V, my_ic:SOT23-5
- added R1, R18: 1k, my_rcl:1608
- C10: value 0.1u -> 10u; device my_rcl:1005 -> my_rcl:2012
- C11: device my_rcl:1608 -> my_rcl:1005
- C24, C25: value 0.1u -> 22p; device my_rcl:1005 -> my_rcl:1608
- C26: value 0.1u -> 10u
- C29, C8: value 0.1u -> 10u; device my_rcl:1608 -> my_rcl:2012
- C30: value 10u -> 0.1u
- C6: device my_rcl:2012 -> my_rcl:1608
- CON1: value USB-A -> MEZZANINE_2X30; device my_connector:UX60A-MB-5ST -> my_connector:MEZZANINE_0.8MM_2X30
- CON3: value MEZZANINE_2X30 -> USB-SC; device my_connector:MEZZANINE_0.8MM_2X30 -> my_connector:UX60SC-MB-5ST
- D1: value LED0 -> USB; device my_rcl:D1608 -> my_rcl:SOD123
- D2: value LED1 -> LED0
- D3: value LED2 -> LED1
- FB1: value FB -> 3.3V
- FB2: value FB -> 1.0V
- IC2: value 1.8V -> MPM3804; device my_ic:SOT23-5 -> my_ic:QFN-10
- R12: value 1k -> 10k
- R13: value 12.1k -> 1k
- R14: value 1k -> 12.1k
- R2: value 10k -> 1k
- moved C28 63.7 mm to (-12.4, -9.40), flipped to the bottom
- moved C26 57.6 mm to (-20.0, -12.4), turned to 270 degrees
- moved C8 54.9 mm to (-23.2, -12.4), turned to 270 degrees
- moved C4 50.1 mm to (-28.4, -13.6), flipped to the bottom, turned to 180 degrees
- moved C27 49.6 mm to (-22.0, -2.00), flipped to the bottom, turned to 180 degrees
- moved C3 44.0 mm to (-24.4, -7.00), flipped to the bottom, turned to 180 degrees
- moved C11 40.2 mm to (-19.2, 8.40), flipped to the bottom
- moved C16 38.5 mm to (-15.6, 5.60), turned to 270 degrees
- moved C6 37.5 mm to (-31.4, -12.4)
- moved CON1 34.8 mm to (-32.4, 8.80), flipped to the bottom, turned to 270 degrees
- moved FB2 32.4 mm to (-25.4, -12.4), turned to 90 degrees
- moved C30 32.0 mm to (-22.0, 19.2), flipped to the bottom
- moved C7 31.4 mm to (-26.4, -9.40), turned to 180 degrees
- moved CON2 28.0 mm to (-4.40, 8.80)
- moved R7 26.9 mm to (-25.8, -0.80), turned to 180 degrees
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- renumbered X2 to X1
Connections:
- removed net LDO1V0: C4.1, IC3.1, IC3.3, J2.2
- removed net LDO1V8: C3.1, IC2.1, IC2.3, J1.2
- removed net N$2 (its old number): D1.K, R15.2
- removed net VCCIO0: C27.1, IC5.3, IC5.7, IC5.8
- new net +1V0_LDO: C5.1, FB2.1, IC3.5
- new net +1V8_DCDC: C6.1, FB3.1, IC2.6, IC2.7, IC2.8, R1.2
- new net +3.3V_LDO: C4.1, FB1.1, IC1.5
- new net N$4: D4.K, R18.2
- new net N$7: IC2.9, R1.1, R2.2
- new net VIN: C1.1, C2.1, CON2.57, CON2.58, CON2.59, CON2.60, D1.2, IC1.1, IC1.3, IC2.1, IC2.5
- net +1V0: now also C9.1, FB2.2; no longer C7.1, IC3.5
- net +1V8: now also C11.1, C19.1, C3.1, CON1.55, CON1.56, CON2.45, CON2.46, CON2.47, CON2.48, FB3.2, FB5.2, FB6.1, IC3.1, IC3.3; no longer C16.1, C26.1, C28.1, C29.1, C6.1, FB2.2, IC2.5
- net +3V3: now also C16.1, C17.1, C18.1, C7.1, CON1.59, CON1.60, CON2.49, CON2.50, CON2.51, CON2.52, FB1.2, FB4.1, IC5.3, IC5.7, IC5.8, R11.2, R4.2; no longer C11.1, C24.1, C25.1, C34.1, C35.1, FB1.1, J1.1, J2.1, R2.2, R5.2
- net ADC_DN1: now also CON1.30; no longer CON2.30
- net ADC_DP1: now also CON1.28; no longer CON2.28
- net DONE: now also R10.1; no longer R9.1
- net DRAM_+1V8: now also C29.1, C30.1, FB5.1; no longer C36.1, FB2.1
- net FLASH_CS: now also R11.1; no longer R10.1
- net FT_+1V8: now also C26.1, C27.1, C28.1, FB6.2; no longer C33.1, IC7.43
- net FT_+3V3: now also C20.1, C21.1, C22.1, C23.1, FB4.2, R12.1, R15.1; no longer C30.1, FB1.2, IC7.44, R11.1, R14.1
- net GND: now also C1.2, C17.2, C18.2, C19.2, C2.2, C20.2, C21.2, C22.2, C23.2, C5.2, C9.2, CON1.1, CON1.2, CON1.31, CON1.32, CON1.52, CON1.53, CON1.54, CON1.57, CON1.58, CON2.14, CON2.15, CON2.16, CON2.33, CON2.34, CON2.35, CON2.36, CON2.37, CON2.38, CON2.39, CON2.40, CON2.41, CON2.42, CON2.43, CON2.44, CON2.53, CON2.54, CON2.55, CON2.56, CON3.5, CON3.M1, CON3.M2, IC1.2, IC2.10, R14.2, R18.1, R2.1, R5.1; no longer C31.2, C32.2, C33.2, C34.2, C35.2, C36.2, CON1.5, CON1.M1, CON1.M2, CON1.M3, CON1.M4, CON2.31, CON2.32, CON3.1, CON3.14, CON3.15, CON3.16, CON3.2, IC2.2, R13.2, R15.1, R4.1
- net INITN: now also R8.1; no longer R7.1
- net IOH0: now also CON1.50; no longer CON2.50
- net IOH1: now also CON1.48; no longer CON2.48
- net IOH10: now also CON1.39; no longer CON2.39
- net IOH100: now also CON2.18; no longer CON3.18
- net IOH101: now also CON2.20; no longer CON3.20
- net IOH102: now also CON2.22; no longer CON3.22
- net IOH103: now also CON2.24; no longer CON3.24
- net IOH104: now also CON2.26; no longer CON3.26
- net IOH105: now also CON2.28; no longer CON3.28
- net IOH106: now also CON2.17; no longer CON3.17
- net IOH107: now also CON2.19; no longer CON3.19
- net IOH108: now also CON2.21; no longer CON3.21
- net IOH109: now also CON2.23; no longer CON3.23
- net IOH11: now also CON1.37; no longer CON2.37
- net IOH110: now also CON2.25; no longer CON3.25
- net IOH111: now also CON2.27; no longer CON3.27
- net IOH112: now also CON2.29; no longer CON3.29
- net IOH113: now also CON2.31; no longer CON3.31
- net IOH114: now also CON2.30; no longer CON3.30
- net IOH115: now also CON2.32; no longer CON3.32
- net IOH12: now also CON1.35; no longer CON2.35
- net IOH13: now also CON1.33; no longer CON2.33
- net IOH14: now also CON1.47; no longer CON2.47
- net IOH15: now also CON1.51; no longer CON2.51
- net IOH16: now also CON1.49; no longer CON2.49
- net IOH17: now also CON1.40; no longer CON2.40
- net IOH18: now also CON1.42; no longer CON2.42
- net IOH2: now also CON1.46; no longer CON2.46
- net IOH3: now also CON1.44; no longer CON2.44
- net IOH4: now also CON1.38; no longer CON2.38
- net IOH5: now also CON1.36; no longer CON2.36
- net IOH6: now also CON1.34; no longer CON2.34
- net IOH7: now also CON1.45; no longer CON2.45
- net IOH8: now also CON1.43; no longer CON2.43
- net IOH9: now also CON1.41; no longer CON2.41
- net IOL0: now also CON1.26; no longer CON2.26
- net IOL1: now also CON1.24; no longer CON2.24
- net IOL10: now also CON1.6; no longer CON2.6
- net IOL101: now also CON2.4; no longer CON3.4
- net IOL102: now also CON2.6; no longer CON3.6
- net IOL103: now also CON2.8; no longer CON3.8
- net IOL104: now also CON2.3; no longer CON3.3
- net IOL105: now also CON2.5; no longer CON3.5
- net IOL106: now also CON2.7; no longer CON3.7
- net IOL107: now also CON2.9; no longer CON3.9
- net IOL108: now also CON2.10; no longer CON3.10
- net IOL109: now also CON2.12; no longer CON3.12
- net IOL11: now also CON1.29; no longer CON2.29
- net IOL110: now also CON2.11; no longer CON3.11
- net IOL111: now also CON2.13; no longer CON3.13
- net IOL12: now also CON1.27; no longer CON2.27
- net IOL13: now also CON1.25; no longer CON2.25
- net IOL14: now also CON1.23; no longer CON2.23
- net IOL15: now also CON1.21; no longer CON2.21
- net IOL16: now also CON1.19; no longer CON2.19
- net IOL17: now also CON1.17; no longer CON2.17
- net IOL18: now also CON1.15; no longer CON2.15
- net IOL19: now also CON1.13; no longer CON2.13
- net IOL2: now also CON1.22; no longer CON2.22
- net IOL20: now also CON1.4; no longer CON2.4
- net IOL21: now also CON1.11; no longer CON2.11
- net IOL22: now also CON1.9; no longer CON2.9
- net IOL23: now also CON1.7; no longer CON2.7
- net IOL24: now also CON1.5; no longer CON2.5
- net IOL25: now also CON1.3; no longer CON2.3
- net IOL3: now also CON1.20; no longer CON2.20
- net IOL4: now also CON1.18; no longer CON2.18
- net IOL5: now also CON1.16; no longer CON2.16
- net IOL6: now also CON1.14; no longer CON2.14
- net IOL7: now also CON1.12; no longer CON2.12
- net IOL8: now also CON1.10; no longer CON2.10
- net IOL9: now also CON1.8; no longer CON2.8
- net JTAG_EN: now also R7.1; no longer R6.1
- net JTAG_TCK: now also R5.2; no longer R4.2
- net JTAG_TDI: now also R4.1; no longer R3.1
- net JTAG_TDO: now also R3.1; no longer R2.1
- net JTAG_TMS: now also R6.1; no longer R5.1
- net LED0: now also D2.A; no longer D1.A
- net LED1: now also D3.A; no longer D2.A
- net LED2: now also D4.A; no longer D3.A
- net N$11: now also R13.2; no longer R12.2
- net N$12: now also R12.2, R13.1; no longer R11.2, R12.1
- net N$13: now also C25.1; no longer C32.1
- net N$14: now also C24.1; no longer C31.1
- net N$15: now also R14.1; no longer R13.1
- net N$16: now also R15.2; no longer R14.2
- net PROGRAMN: now also R9.1; no longer R8.1
- net USB_+5V: now also CON3.1, D1.1; no longer CON1.1
- net USB_DM: now also CON3.2; no longer CON1.2
- net USB_DP: now also CON3.3; no longer CON1.3
Routing:
- net +3V3: track 32.2 -> 141.0 mm, vias 5 -> 9
- net VIN: track 0.00 -> 74.6 mm, vias 0 -> 3
- net +1V8: track 64.9 -> 138.2 mm, vias 15 -> 20
- net +1V8_DCDC: track 0.00 -> 12.6 mm, vias 0 -> 1
- net N$11: track 13.6 -> 7.56 mm, vias 0 -> 1
- net FT_+3V3: track 39.5 -> 45.5 mm, vias 7 -> 8
- net DRAM_+1V8: track 12.8 -> 18.6 mm, vias 4 -> 6
- net +1V0: track 40.7 -> 35.4 mm
- net USB_+5V: track 0.00 -> 4.40 mm, vias 0 -> 1
- net +3.3V_LDO: track 0.00 -> 3.87 mm, vias 0 -> 1
- net N$7: track 0.00 -> 3.29 mm, vias 0 -> 1
- net GND: track 1.93 -> 5.01 mm, vias 21 -> 22
- net FT_+1V8: track 22.4 -> 25.0 mm
- net +1V0_LDO: track 0.00 -> 2.06 mm, vias 0 -> 1
- net N$4: track 0.00 -> 1.80 mm
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- added copper zone on layer 1, net GND
- added copper zone on layer 15, net GND
- added copper zone on layer 16, net GND
Other:
- board outline added: 40 x 40 mm
- board text added: "FPGA Core Board ver1"

Commit message: 6層
Parts:
- added C31, C32: 10u, my_rcl:1608
- added C33, C34: 0.1u, my_rcl:1608
- added FB7: VIN, my_rcl:1608-J
- C4, C5: value 0.1u -> 1u
- R1: value 1k -> 10k
- R2: value 1k -> 5k
- moved D1 0.80 mm to (-5.20, -8.40)
- moved C29 0.40 mm to (-13.2, 19.2)
- moved C28 0.20 mm to (-12.2, -9.40)
Connections:
- new net 1.8V_DCDC_SW: IC2.2, IC2.3, IC2.4
- new net VIN_DCDC: C1.1, C2.1, C31.1, C32.1, FB7.2, IC1.1, IC1.3, IC2.1, IC2.5
- net DRAM_+1V8: now also C33.1
- net GND: now also C31.2, C32.2, C33.2, C34.2
- net VIN: now also C34.1, FB7.1; no longer C1.1, C2.1, IC1.1, IC1.3, IC2.1, IC2.5
Routing:
- net +1V8: track 138.2 -> 241.4 mm, vias 20 -> 24
- net +3V3: track 141.0 -> 216.4 mm, vias 9 -> 11
- net FT_+3V3: track 45.5 -> 72.3 mm
- net VIN_DCDC: track 0.00 -> 24.9 mm, vias 0 -> 3
- net VIN: track 74.6 -> 95.6 mm, vias 3 -> 4
- net FT_+1V8: track 25.0 -> 45.0 mm
- net +1V0: track 35.4 -> 50.6 mm
- net 1.8V_DCDC_SW: track 0.00 -> 2.35 mm
- net +1V8_DCDC: track 12.6 -> 14.6 mm
- net GND: track 5.01 -> 6.94 mm
- net USB_+5V: track 4.40 -> 3.60 mm
- net DRAM_+1V8: track 18.6 -> 18.5 mm, vias 6 -> 7
- added copper zone on layer 14, net GND
- added copper zone on layer 3, net GND

Commit message: 発注
Parts:
- added C35: 0.1u, my_rcl:1608
- added J1: CLK, my_rcl:1608-J
- added X2: 12MHz, my_rcl:KC3225
- C11, C13: value 0.1u -> 10u; device my_rcl:1005 -> my_rcl:2012
- C18, C21, C23: device my_rcl:1608 -> my_rcl:1005
- C19: device my_rcl:1005 -> my_rcl:1608
- C20: value 10u -> 0.1u; device my_rcl:1608 -> my_rcl:1005
- C24: value 22p -> 10u
- C25: value 22p -> 0.1u
- C26, C31, C32, C6: value 10u -> 0.1u
- C28: value 0.1u -> 22p
- C29: value 10u -> 22p; device my_rcl:2012 -> my_rcl:1608
- C3, C30: value 0.1u -> 10u
- C34: value 0.1u -> 10u; device my_rcl:1608 -> my_rcl:2012
- C4: value 1u -> 0.1u
- C5: value 1u -> 10u
- C7, C8: value 10u -> 1u; device my_rcl:2012 -> my_rcl:1608
- C9: value 0.1u -> 10u; device my_rcl:1005 -> my_rcl:1608
- FB1: value 3.3V -> VIN
- FB2: value 1.0V -> 3.3V
- FB3: value 1.8V -> 1.0V
- FB4: value FT -> 1.8V
- FB5: value DRAM -> FT
- FB7: value VIN -> DRAM
- IC8: value HYPERRAM -> HyperRAM
- X1: value 12MHz -> 25MHz
- moved C30 31.7 mm to (-20.0, -12.4), flipped to the top
- moved FB7 29.9 mm to (-25.2, 19.6), flipped to the top, turned to 270 degrees
- moved C34 29.4 mm to (-13.2, 19.2), flipped to the top, turned to 90 degrees
- moved FB5 28.5 mm to (-23.4, -8.80), turned to 90 degrees
- moved C29 27.6 mm to (-9.60, -8.20), turned to 180 degrees
- moved C9 25.4 mm to (-31.4, -12.4), flipped to the top, turned to 90 degrees
- moved C1 25.2 mm to (-3.20, -8.40), turned to 270 degrees
- moved C13 24.7 mm to (-29.4, -8.80), flipped to the top, turned to 90 degrees
- moved C32 21.2 mm to (-12.2, -9.40), turned to 0 degrees
- moved C11 21.2 mm to (-23.2, -12.4), flipped to the top, turned to 270 degrees
- moved C18 20.7 mm to (-23.6, 16.0), flipped to the bottom, turned to 180 degrees
- moved C20 18.2 mm to (-15.6, 5.60), flipped to the bottom
- moved C31 15.4 mm to (-22.0, -2.00), turned to 180 degrees
- moved C19 14.4 mm to (-9.60, 0.80), turned to 270 degrees
- moved C22 13.9 mm to (-5.20, 6.60), flipped to the top
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Connections:
- new net N$6: J1.1, X1.3
- net +1V0: now also C11.1, C15.1, C17.1, FB3.2; no longer C14.1, C8.1, C9.1, FB2.2
- net +1V0_LDO: now also C8.1, FB3.1; no longer C5.1, FB2.1
- net +1V8: now also C14.1, C16.1, C18.1, C23.1, C6.1, FB4.2, FB7.2; no longer C10.1, C11.1, C15.1, C19.1, C3.1, FB3.2, FB5.2
- net +1V8_DCDC: now also C9.1, FB4.1; no longer C6.1, FB3.1
- net +3.3V_LDO: now also C7.1, FB2.1; no longer C4.1, FB1.1
- net +3V3: now also C10.1, C19.1, C20.1, C21.1, C22.1, FB2.2, FB5.1, X1.1, X1.4; no longer C16.1, C17.1, C18.1, C7.1, FB1.2, FB4.1
- net DRAM_+1V8: now also C34.1, C35.1, FB7.1; no longer C29.1, C30.1, FB5.1
- net FT_+1V8: now also C30.1, C31.1, C32.1; no longer C26.1, C27.1, C28.1
- net FT_+3V3: now also C24.1, C25.1, C26.1, C27.1, FB5.2; no longer C20.1, C21.1, C22.1, C23.1, FB4.2
- net GND: now also C35.2, X2.2, X2.4; no longer X1.4
- net IOH112: now also J1.2
- net N$13: now also C29.1, X2.3; no longer C25.1, X1.3
- net N$14: now also C28.1, X2.1; no longer C24.1, X1.1
- net VIN: now also C1.1, FB1.1; no longer C34.1, FB7.1
- net VIN_DCDC: now also C3.1, C4.1, C5.1, FB1.2; no longer C1.1, C31.1, C32.1, FB7.2
Routing:
- net +3V3: track 216.4 -> 223.2 mm
- net IOH112: track 13.6 -> 16.0 mm, vias 1 -> 2
- net N$6: track 0.00 -> 1.59 mm
- net FT_+1V8: track 45.0 -> 45.7 mm
- net +1V8: track 241.4 -> 242.0 mm
- net VIN: track 95.6 -> 96.2 mm
- net GND: vias 22 -> 142

Commit message: コネクタをピン名に変更
Connections:
- net IOH0 renamed PR24B
- net IOH1 renamed PR27A
- net IOH10 renamed PR27B
- net IOH100 renamed PL44B
- net IOH101 renamed PL44A
- net IOH102 renamed PL38B
- net IOH103 renamed PL38A
- net IOH104 renamed PL26B
- net IOH105 renamed PL26A
- net IOH106 renamed PL42B
- net IOH107 renamed PL42A
- net IOH108 renamed PL36B
- net IOH109 renamed PL36A
- net IOH11 renamed PR32B
- net IOH110 renamed PL32B
- net IOH111 renamed PL32A
- net IOH112 renamed PL30A
- net IOH113 renamed PL30B
- net IOH114 renamed PL24A
- net IOH115 renamed PL24B
- net IOH12 renamed PR42A
- net IOH13 renamed PR42B
- net IOH14 renamed PR26A
- net IOH15 renamed PR13B
- net IOH16 renamed PR17A
- net IOH17 renamed PR34A
- net IOH18 renamed PR36B
- net IOH2 renamed PR24A
- net IOH3 renamed PR36A
- net IOH4 renamed PR34B
- net IOH5 renamed PR38B
- net IOH6 renamed PR38A
- net IOH7 renamed PR30A
- net IOH8 renamed PR32A
- net IOH9 renamed PR30B
- net IOL0 renamed PB84A
- net IOL1 renamed PB84B
- net IOL10 renamed PB74B
- net IOL101 renamed PB12B
- net IOL102 renamed PB12A
- net IOL103 renamed PB8B
- net IOL104 renamed PB10B
- net IOL105 renamed PB8A
- net IOL106 renamed PB10A
- net IOL107 renamed PB4B
- net IOL108 renamed PB6B
- net IOL109 renamed PB6A
- net IOL11 renamed PB66A
- net IOL110 renamed PL47A
- net IOL111 renamed PB4A
- net IOL12 renamed PB66B
- net IOL13 renamed PB70A
- net IOL14 renamed PB70B
- net IOL15 renamed PB64B
- net IOL16 renamed PB68B
- net IOL17 renamed PB64A
- net IOL18 renamed PB68A
- net IOL19 renamed PB72B
- net IOL2 renamed PB82B
- net IOL20 renamed PB74A
- net IOL21 renamed PB72A
- net IOL22 renamed PB60B
- net IOL23 renamed PB60A
- net IOL24 renamed PB58B
- net IOL25 renamed PB58A
- net IOL3 renamed PB82A
- net IOL4 renamed PB80B
- net IOL5 renamed PB80A
- net IOL6 renamed PB78A
- net IOL7 renamed PB78B
- net IOL8 renamed PB76B
- net IOL9 renamed PB76A
