File: ADC3_FPGA_BGA.brd (EAGLE design)
At the start: 40 x 40 mm, 80 parts, among them CON1 MEZZANINE_2X30, CON2 MEZZANINE_2X30, CON3 USB-SC, IC1 3.3V, IC2 MPM3804, IC3 1.0V, IC4 LFD2NX-40, IC5 EEPROM, IC6 93LC56, IC7 FT2232H, IC8 HyperRAM, J1 CLK, X1 25MHz, X2 12MHz

Commit message: FT2232のEEPROMの配線を修正
Parts:
- moved R12 0.40 mm to (-15.0, -11.6)
- moved R13 0.40 mm to (-15.0, -13.4)
Connections:
- net N$10: now also R13.2
- net N$11: no longer R13.2
Routing:
- net N$10: track 5.24 -> 7.81 mm, vias 0 -> 1
- net N$11: track 7.56 -> 5.73 mm, vias 1 -> 0
Changed lines of the file:
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@@
 <attribute name="NAME" x="-6.68" y="-4.355" size="0.8128" layer="25" rot="R270"/>
 </element>
-<element name="R13" library="my_rcl" package="1608" value="1k" x="-14.6" y="-13.4" smashed="yes" rot="MR180">
-<attribute name="NAME" x="-16.2" y="-14.4" size="0.8128" layer="26" rot="MR180"/>
-<attribute name="VALUE" x="-17.6" y="-12.8" size="0.8128" layer="28" font="vector" ratio="15" rot="MR180"/>
-</element>
-<element name="R12" library="my_rcl" package="1608" value="10k" x="-14.6" y="-11.6" smashed="yes" rot="MR0">
-<attribute name="NAME" x="-13" y="-10.6" size="0.8128" layer="26" rot="MR0"/>
-<attribute name="VALUE" x="-18.4" y="-11.2" size="0.8128" layer="28" font="vector" ratio="15" rot="MR180"/>
+<element name="R13" library="my_rcl" package="1608" value="1k" x="-15" y="-13.4" smashed="yes" rot="MR180">
+<attribute name="NAME" x="-16.6" y="-14.4" size="0.8128" layer="26" rot="MR180"/>
+<attribute name="VALUE" x="-13.2" y="-13.4" size="0.8128" layer="28" font="vector" ratio="15" rot="MR180"/>
+</element>
+<element name="R12" library="my_rcl" package="1608" value="10k" x="-15" y="-11.6" smashed="yes" rot="MR0">
+<attribute name="NAME" x="-13.4" y="-10.6" size="0.8128" layer="26" rot="MR0"/>
+<attribute name="VALUE" x="-13.2" y="-11.6" size="0.8128" layer="28" font="vector" ratio="15" rot="MR180"/>
 </element>
 <element name="IC6" library="my_ic" package="SOT23-6" value="93LC56" x="-14.8" y="-12.8" smashed="yes" rot="R270">
@@
 <element name="C32" library="my_rcl" package="1608" value="0.1u" x="-12.2" y="-9.4" smashed="yes" rot="MR0">
 <attribute name="NAME" x="-10.6" y="-8.4" size="0.8128" layer="26" rot="MR0"/>
-<attribute name="VALUE" x="-10.2" y="-11.2" size="0.8128" layer="28" font="vector" ratio="15" rot="MR0"/>
+<attribute name="VALUE" x="-10.4" y="-11.2" size="0.8128" layer="28" font="vector" ratio="15" rot="MR0"/>
 </element>
 <element name="C27" library="my_rcl" package="1608" value="0.1u" x="-12.8" y="-1.2" smashed="yes" rot="MR270">
@@
 <wire x1="-13.4" y1="-10.4" x2="-13.4" y2="-10.8" width="0.254" layer="1"/>
 <wire x1="-13.4" y1="-10.8" x2="-13" y2="-11.2" width="0.254" layer="1"/>
-<wire x1="-13.5" y1="-11.2" x2="-13.7" y2="-11.4" width="0.254" layer="16"/>
-<wire x1="-13.7" y1="-11.6" x2="-13.7" y2="-11.4" width="0.254" layer="16"/>
-<wire x1="-13.5" y1="-11.2" x2="-13" y2="-11.2" width="0.254" layer="16"/>
+<wire x1="-13.7" y1="-11.2" x2="-14.1" y2="-11.6" width="0.254" layer="16"/>
+<wire x1="-13.7" y1="-11.2" x2="-13" y2="-11.2" width="0.254" layer="16"/>
 <wire x1="-13.5" y1="-11.85" x2="-13.25" y2="-11.85" width="0.254" layer="1"/>
 <wire x1="-13.25" y1="-11.85" x2="-13" y2="-11.6" width="0.254" layer="1"/>
@@
 <wire x1="-16.1" y1="-13.75" x2="-15.75" y2="-13.75" width="0.127" layer="1"/>
 <wire x1="-15.75" y1="-13.75" x2="-15" y2="-13" width="0.127" layer="1"/>
-<wire x1="-15" y1="-13" x2="-15" y2="-11" width="0.127" layer="1"/>
+<wire x1="-15" y1="-13" x2="-15" y2="-11.2" width="0.127" layer="1"/>
+<contactref element="R13" pad="2"/>
+<wire x1="-15" y1="-11.2" x2="-15" y2="-11" width="0.127" layer="1"/>
+<wire x1="-14.1" y1="-13.4" x2="-14.1" y2="-13.1" width="0.1524" layer="16"/>
+<wire x1="-15" y1="-12.2" x2="-15" y2="-11.2" width="0.1524" layer="16"/>
+<via x="-15" y="-11.2" extent="1-16" drill="0.35"/>
+<wire x1="-14.1" y1="-13.1" x2="-15" y2="-12.2" width="0.1524" layer="16"/>
 </signal>
 <signal name="N$11">
 <contactref element="IC7" pad="1"/>
-<contactref element="R13" pad="2"/>
 <contactref element="IC6" pad="5"/>
 <wire x1="-13" y1="-8.45" x2="-12.55" y2="-8.45" width="0.127" layer="1"/>
@@
 <wire x1="-12.4" y1="-12.4" x2="-12.8" y2="-12.8" width="0.127" layer="1"/>
 <wire x1="-13.5" y1="-12.8" x2="-12.8" y2="-12.8" width="0.127" layer="1"/>
-<via x="-12.4" y="-12.4" extent="1-16" drill="0.3"/>
-<wire x1="-12.4" y1="-12.4" x2="-13" y2="-13" width="0.127" layer="16"/>
-<wire x1="-13" y1="-13" x2="-13.5" y2="-13" width="0.127" layer="16"/>
-<wire x1="-13.5" y1="-13" x2="-13.7" y2="-13.2" width="0.127" layer="16"/>
-<wire x1="-13.7" y1="-13.2" x2="-13.7" y2="-13.4" width="0.127" layer="16"/>
 </signal>
 <signal name="N$12">
@@
 <contactref element="R12" pad="2"/>
 <contactref element="IC6" pad="1"/>
-<wire x1="-16.1" y1="-11.85" x2="-16.95" y2="-11.85" width="0.127" layer="1"/>
+<wire x1="-16.2" y1="-11.85" x2="-16.95" y2="-11.85" width="0.127" layer="1"/>
 <wire x1="-16.95" y1="-11.85" x2="-17" y2="-11.8" width="0.127" layer="1"/>
 <via x="-17" y="-11.8" extent="1-16" drill="0.3"/>
-<wire x1="-17" y1="-11.8" x2="-15.7" y2="-11.8" width="0.127" layer="16"/>
-<wire x1="-15.7" y1="-11.8" x2="-15.5" y2="-11.6" width="0.127" layer="16"/>
-<wire x1="-15.5" y1="-13.4" x2="-15.5" y2="-11.6" width="0.127" layer="16"/>
+<wire x1="-17" y1="-11.8" x2="-16.1" y2="-11.8" width="0.127" layer="16"/>
+<wire x1="-16.1" y1="-11.8" x2="-15.9" y2="-11.6" width="0.127" layer="16"/>
+<wire x1="-15.9" y1="-11.6" x2="-15.9" y2="-13.4" width="0.127" layer="16"/>
+<wire x1="-16.1" y1="-11.85" x2="-16.2" y2="-11.85" width="0.1524" layer="1"/>
 </signal>
 <signal name="N$13">
@@
 <contactref element="IC6" pad="4"/>
 <contactref element="IC7" pad="56"/>
-<wire x1="-13.95" y1="-9.4" x2="-13.95" y2="-10.55" width="0.127" layer="1"/>
+<wire x1="-13.95" y1="-9.4" x2="-13.95" y2="-10.95" width="0.127" layer="1"/>
 <wire x1="-13.85" y1="-13.75" x2="-13.5" y2="-13.75" width="0.127" layer="1"/>
-<wire x1="-13.95" y1="-10.55" x2="-14.6" y2="-11.2" width="0.127" layer="1"/>
-<wire x1="-14.6" y1="-11.2" x2="-14.6" y2="-13" width="0.127" layer="1"/>
+<wire x1="-13.95" y1="-10.95" x2="-14.6" y2="-11.6" width="0.127" layer="1"/>
+<wire x1="-14.6" y1="-11.6" x2="-14.6" y2="-13" width="0.127" layer="1"/>
 <wire x1="-14.6" y1="-13" x2="-13.85" y2="-13.75" width="0.127" layer="1"/>
 </signal>
