File: ADC3_FPGA_BGA.brd (EAGLE design)
At the start: 40.4 x 44.4 mm, 115 parts, among them CON1 MEZZANINE_2X30, CON2 MEZZANINE_2X30, CON3 USB-C, IC1 ARTIX7-FTG256, IC2 3.3V, IC3 2.5V, IC4 MPM3804, IC5 MPM3804, IC6 EEPROM, IC7 93LC56, IC8 FT2232H, IC9 HyperRAM, J1 BANK34, J2 BANK35, J3 25M, X1 25MHz, X2 12MHz

Commit message: 発注
Parts:
- added C30, C58: 0.1u, my_rcl:1608C
- IC4: value MPM3804 -> MPM3811
- moved C29 1.75 mm to (-9.00, 13.5)
- moved CON3 0.50 mm to (13.5, -20.2)
- turned CON2 to 90 degrees
Connections:
- net +1V8: now also C30.1, C58.1, CON2.13, CON2.14, CON2.15, CON2.16; no longer CON2.45, CON2.46, CON2.47, CON2.48
- net +3V3: now also CON2.10, CON2.11, CON2.12, CON2.9; no longer CON2.49, CON2.50, CON2.51, CON2.52
- net GND: now also C30.2, C58.2, CON2.17, CON2.18, CON2.19, CON2.20, CON2.37, CON2.38, CON2.5, CON2.59, CON2.6, CON2.60, CON2.7, CON2.8; no longer CON2.1, CON2.2, CON2.23, CON2.24, CON2.41, CON2.42, CON2.43, CON2.44, CON2.53, CON2.54, CON2.55, CON2.56
- net IO0_14: now also CON2.35; no longer CON2.26
- net IO10N_15: now also CON2.54; no longer CON2.7
- net IO10P_15: now also CON2.52; no longer CON2.9
- net IO11N_14: now also CON2.21; no longer CON2.40
- net IO11P_14: now also CON2.23; no longer CON2.38
- net IO12N_14: now also CON2.29; no longer CON2.32
- net IO12P_14: now also CON2.31; no longer CON2.30
- net IO13N_15: now also CON2.49; no longer CON2.12
- net IO13P_15: now also CON2.47; no longer CON2.14
- net IO15N_15: now also CON2.51; no longer CON2.10
- net IO15P_15: now also CON2.53; no longer CON2.8
- net IO17N_15: now also CON2.50; no longer CON2.11
- net IO17P_15: now also CON2.48; no longer CON2.13
- net IO21N_15: now also CON2.45; no longer CON2.16
- net IO21P_15: now also CON2.43; no longer CON2.18
- net IO22N_15: now also CON2.46; no longer CON2.15
- net IO22P_15: now also CON2.44; no longer CON2.17
- net IO23N_15: now also CON2.40; no longer CON2.21
- net IO23P_15: now also CON2.42; no longer CON2.19
- net IO24N_15: now also CON2.41; no longer CON2.20
- net IO24P_15: now also CON2.39; no longer CON2.22
- net IO2N_14: now also CON2.34; no longer CON2.27
- net IO2P_14: now also CON2.36; no longer CON2.25
- net IO4N_14: now also CON2.30; no longer CON2.31
- net IO4P_14: now also CON2.32; no longer CON2.29
- net IO5P_14: now also CON2.33; no longer CON2.28
- net IO7N_14: now also CON2.26; no longer CON2.35
- net IO7P_14: now also CON2.28; no longer CON2.33
- net IO8N_14: now also CON2.22; no longer CON2.39
- net IO8N_15: now also CON2.57; no longer CON2.4
- net IO8P_14: now also CON2.24; no longer CON2.37
- net IO8P_15: now also CON2.55; no longer CON2.6
- net IO9N_14: now also CON2.25; no longer CON2.36
- net IO9N_15: now also CON2.58; no longer CON2.3
- net IO9P_14: now also CON2.27; no longer CON2.34
- net IO9P_15: now also CON2.56; no longer CON2.5
- net VIN: now also CON2.1, CON2.2, CON2.3, CON2.4; no longer CON2.57, CON2.58, CON2.59, CON2.60
Routing:
- net +1V8: track 35.3 -> 42.0 mm, vias 17 -> 20
- net +3V3: track 63.0 -> 65.2 mm, vias 25 -> 24
- net GND: track 4.14 -> 6.22 mm, vias 156 -> 161
- net VIN: track 38.6 -> 40.1 mm, vias 3 -> 4
- net USB_DM: track 13.8 -> 13.2 mm
- net N$6: track 12.2 -> 11.6 mm
Other:
- board text added: "FPGA Core Board ver3"
- board text removed: "FPGA Core Board ve3"

Commit message: 微修正
Parts:
- removed D6: P, my_rcl:D1608
- added C59, C60: 1u, my_rcl:1608C
- added C61: 10u, my_rcl:2012
- added D1: 0, my_rcl:D1608
- C10, C44, C45, C47: value 0.1u -> 1u; device my_rcl:1608C -> my_rcl:1005
- C11, C7, C8: value 1u -> 4.7u; device my_rcl:1005 -> my_rcl:1608C
- C17, C18, C46: value 10u -> 1u; device my_rcl:1608C -> my_rcl:1005
- C21, C22: value 10u -> 1u; device my_rcl:2012 -> my_rcl:1005
- C23, C24: device my_rcl:2012 -> my_rcl:1608C
- C29: device my_rcl:3216 -> my_rcl:2012
- C30: value 0.1u -> 10u; device my_rcl:1608C -> my_rcl:2012
- C31: value 1u -> 10u; device my_rcl:1005 -> my_rcl:3216
- C32, C33: value 1u -> 10u; device my_rcl:1005 -> my_rcl:2012
- C34, C5, C6: value 1u -> 0.1u; device my_rcl:1005 -> my_rcl:1608C
- C50: value 22p -> 10u
- C51: value 22p -> 0.1u
- C52: value 10u -> 0.1u
- C54, C55: value 0.1u -> 22p
- C56: value 0.1u -> 10u
- C57: value 10u -> 0.1u; device my_rcl:2012 -> my_rcl:1608C
- C9: value 0.1u -> 4.7u
- D2: value 0 -> 1
- D3: value 1 -> 2
- D4: value 2 -> 3
- D5: value 3 -> P
- FB1: value VIN -> USB
- FB2: value 3.3V -> VIN
- FB3: value 2.5V -> 3.3V
- FB4: value 1.8V -> 2.5V
- FB5: value 1.0V -> 1.8V
- FB6: value FT -> 1.0V
- FB8: value DRAM -> FT
- FB9: value USB -> DRAM
- R16, R17: value 1k -> 5.1k
- R18: value 12.1k -> 1k
- R20: value 1k -> 12.1k
- R22, R23: value 5.1k -> 1k
- X1: value 25MHz -> OSC
- moved FB9 38.5 mm to (-4.00, 13.0), flipped to the top, turned to 270 degrees
- moved R23 38.1 mm to (-0.50, 16.2), turned to 180 degrees
- moved C9 36.2 mm to (10.8, 13.5), flipped to the top, turned to 270 degrees
- moved C56 33.8 mm to (4.50, -19.8), turned to 0 degrees
- moved C58 33.1 mm to (4.50, -18.0), flipped to the bottom, turned to 0 degrees
- moved C55 31.8 mm to (9.00, -18.0), flipped to the top, turned to 0 degrees
- moved C29 31.7 mm to (-16.8, -17.2), flipped to the bottom, turned to 0 degrees
- moved R21 30.8 mm to (9.00, -13.0), flipped to the top
- moved C30 29.8 mm to (-6.75, -15.2), flipped to the bottom, turned to 180 degrees
- moved C17 27.4 mm to (3.00, 1.50)
- moved C57 27.3 mm to (-1.50, -12.0), flipped to the bottom, turned to 180 degrees
- moved R20 27.3 mm to (9.00, -16.2), turned to 0 degrees
- moved C22 27.1 mm to (-1.00, 2.50), turned to 180 degrees
- moved R22 25.9 mm to (-18.2, -15.0), flipped to the top, turned to 90 degrees
- moved R18 25.5 mm to (-16.5, -15.0), turned to 90 degrees
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Connections:
- net +1V0: now also C10.1, C12.1, C14.1, C18.1, C22.1, C28.1, C30.1, C8.1, FB6.2; no longer C11.1, C13.1, C15.1, C24.1, C26.1, C5.1, C7.1, FB5.2
- net +1V0_DCDC: now also C24.1, FB6.1; no longer C20.1, FB5.1
- net +1V8: now also C11.1, C13.1, C15.1, C17.1, C21.1, C27.1, C31.1, C34.1, C42.1, C44.1, C7.1, C9.1, FB5.2, FB8.1, FB9.2; no longer C12.1, C14.1, C23.1, C25.1, C30.1, C36.1, C38.1, C58.1, C6.1, C8.1, FB4.2, FB7.1, FB8.2
- net +1V8_DCDC: now also C23.1, FB5.1; no longer C19.1, FB4.1
- net +2V5: now also C26.1, FB4.2; no longer C22.1, FB3.2
- net +2V5_LDO: now also C20.1, FB4.1; no longer C18.1, FB3.1
- net +3V3: now also C25.1, C46.1, C47.1, C48.1, C49.1, D5.A, FB3.2, FB7.1; no longer C21.1, C37.1, C39.1, C42.1, C44.1, D6.A, FB2.2, FB6.1
- net +3V3_LDO: now also C19.1, FB3.1; no longer C17.1, FB2.1
- net DRAM_+1V8: now also C59.1, C60.1, C61.1, FB9.1, R23.2; no longer C55.1, C56.1, C57.1, FB8.1, R21.2
- net DRAM_NRST: now also R23.1; no longer R21.1
- net FT_+1V8: now also C56.1, C57.1, C58.1, FB8.2; no longer C52.1, C53.1, C54.1, FB7.2
- net FT_+3V3: now also C50.1, C51.1, C52.1, C53.1, FB7.2, R21.1; no longer C46.1, C47.1, C48.1, C49.1, FB6.2, R19.1
- net GND: now also C59.2, C60.2, C61.2, R17.1, R18.1, R20.2; no longer R18.2, R20.1, R23.1
- net LED0: now also D1.A; no longer D2.A
- net LED1: now also D2.A; no longer D3.A
- net LED2: now also D3.A; no longer D4.A
- net LED3: now also D4.A; no longer D5.A
- net N$1: now also D5.K, R22.2; no longer D6.K, R20.2
- net N$10: now also R19.2; no longer R17.2
- net N$12: now also R19.1; no longer R17.1
- net N$13: now also C55.1; no longer C51.1
- net N$14: now also C54.1; no longer C50.1
- net N$15: now also R20.1; no longer R18.1
- net N$16: now also R21.2; no longer R19.2
- net N$2: now also D1.K; no longer D2.K
- net N$3: now also D2.K; no longer D3.K
- net N$4: now also D3.K; no longer D4.K
- net N$5: now also D4.K, R18.2; no longer D5.K, R16.2
- net N$6: now also R16.2; no longer R22.2
- net N$7: now also R17.2; no longer R23.2
- net USB_+5V: now also FB1.1; no longer FB9.1
- net VCCO34: now also C32.1, C35.1, C37.1; no longer C27.1, C31.1, C33.1
- net VCCO35: now also C33.1, C36.1, C38.1, C39.1; no longer C28.1, C32.1, C34.1, C35.1
- net VIN: now also FB1.2, FB2.1; no longer FB1.1, FB9.2
- net VIN_DCDC: now also C5.1, C6.1, FB2.2; no longer C10.1, C9.1, FB1.2
Routing:
- net +1V8: track 42.0 -> 31.0 mm, vias 20 -> 21
- net +3V3: track 65.2 -> 60.7 mm
- net +1V0: track 7.02 -> 7.74 mm, vias 11 -> 12
- net GND: vias 161 -> 168
