File: ADC3_FPGA_BGA.sch (EAGLE design)
At the start: 129 parts, among them CON1 2X17-FEMALE, IC1 3.3V, IC2 1.8V, IC3 1.0V, IC4 LFD2NX-40, IC5 EEPROM, IC6 AE-FT232HL, J1 SJ-1608, J2 SJ-1608, J3 IO0, J4 IO2, J5 IO6, J6 IO3, J7 IO4, SW1 5V, U1 DC-DC, X1 OSC

Commit message: 発注
Parts:
- added FB3: FB, my_rcl:FB
- added J8: 1.0V, my_rcl:SJ-1608
- added TP23: TX, my_connector:TESTPIN
- added TP24: GND, my_connector:TESTPIN
Connections:
- net CLK_25M renamed CLK_20M
- new net +1V0CORE: C12.1, C14.1, C17.1, C9.1, IC4G$1.VCC, IC4G$1.VCCECLK, J8.2, TP3.1
- new net N$9: FB3.2, SW1.2
- new net UART_TX: IC4G$9.PL4B, TP23.1
- net +1V0: now also J8.1; no longer C12.1, C14.1, C17.1, C9.1, IC4G$1.VCC, IC4G$1.VCCECLK, TP3.1
- net +5V: now also FB3.1; no longer SW1.2
- net GND: now also TP24.1

Commit message: メザニンコネクタ
Parts:
- removed C1, C17, C18, C19, C20, C21, C22, C23, C5: 10u, my_rcl:C-3225
- removed C2, C9: 0.1u, my_rcl:C-1608
- removed D4: LED3, my_rcl:LED-SMD1608
- removed DR1, DR2, DR3, DR4: HOLE-3.2, my_connector:HOLE-3.2
- removed F1: 0.9A, my_rcl:FUSE-3216
- removed FB3: FB, my_rcl:FB
- removed IC1: 3.3V, my_ic:78X-3
- removed J3: IO0, my_rcl:SJ-1608
- removed J4: IO2, my_rcl:SJ-1608
- removed J5: IO6, my_rcl:SJ-1608
- removed J6: IO3, my_rcl:SJ-1608
- removed J7: IO4, my_rcl:SJ-1608
- removed J8: 1.0V, my_rcl:SJ-1608
- removed JP1: JTAG, my_connector:PINHD-1X7
- removed JP2: SPI, my_connector:PINHD-1X7
- removed JP3: LVIO, pinhead:PINHD-2X20
- removed JP4: HVIO, pinhead:PINHD-2X3
- removed R1: 22, my_rcl:R-1608J
- removed R18, R26: D1, my_rcl:R-1608J
- removed R20, R30: D5, my_rcl:R-1608J
- removed R21, R32: D7, my_rcl:R-1608J
- removed R22: D9, my_rcl:R-1608J
- removed R23: D11, my_rcl:R-1608J
- removed R24: D13, my_rcl:R-1608J
- removed R25: D0, my_rcl:R-1608J
- removed R27: D2, my_rcl:R-1608J
- removed R28: D3, my_rcl:R-1608J
- removed R29: D4, my_rcl:R-1608J
- removed R31: D6, my_rcl:R-1608J
- removed R33: CLK, my_rcl:R-1608J
- removed R34: WR, my_rcl:R-1608J
- removed R35: RD, my_rcl:R-1608J
- removed R36: TXNE, my_rcl:R-1608J
- removed R37: RXNF, my_rcl:R-1608J
- removed R38, R39, R40, R41, R42: 1k, my_rcl:R-1608
- removed SW1: 5V, my_connector:SW-1X3
- removed TP1: ADCP, my_connector:TESTPIN-PAD
- removed TP10, TP22, TP24: GND, my_connector:TESTPIN
- removed TP11, TP12, TP13, TP14, TP15, TP16, TP17, TP18: (no value), my_connector:TESTPIN-PAD
- removed TP19: VIN+, my_connector:TESTPIN
- removed TP2: ADCN, my_connector:TESTPIN-PAD
- removed TP20: VIN-, my_connector:TESTPIN
- removed TP21: FT_+5V, my_connector:TESTPIN
- removed TP23: TX, my_connector:TESTPIN
- removed TP3: 1.0V, my_connector:TESTPIN
- removed TP4: 1.8V, my_connector:TESTPIN
- removed TP5: VCCIO0, my_connector:TESTPIN
- removed TP6: VCCIO2, my_connector:TESTPIN
- removed TP7: VCCIO6, my_connector:TESTPIN
- removed TP8: VCCIO3, my_connector:TESTPIN
- removed TP9: VCCIO4, my_connector:TESTPIN
- removed U1: DC-DC, my_ic:DC-DC
- removed X1: OSC, my_rcl:OSC-KC3225
- added C33, C36: 10u, my_rcl:C-1608
- added C34, C35: 0.1u, my_rcl:C-1608
- added CON2, CON3: MEZZANINE_2X30, my_connector:MEZZANINE_2X30
- added IC7: FT2232H, my_ic:FT2232H
- added IC8: HYPERRAM, my_ic:HYPERRAM
- added X2: 12MHz, my_rcl:CRYSTAL2
- C10, C12, C13, C14, C15, C16, C24, C25: device my_rcl:C-1608 -> my_rcl:C-1005
- C30: value 0.1u -> 10u
- C31, C32: value 100u -> 22p; device my_rcl:CPOLE2.5-8 -> my_rcl:C-1608
- CON1: value 2X17-FEMALE -> USB-A; device my_connector:2X17-FEMALE -> my_connector:USB-A
- IC6: value AE-FT232HL -> 93LC56; device my_ic:AE-FT232HL -> my_ic:93LC56
- R11: value D0 -> 10k; device my_rcl:R-1608J -> my_rcl:R-1608
- R12: value D2 -> 1k; device my_rcl:R-1608J -> my_rcl:R-1608
- R13: value D4 -> 12.1k; device my_rcl:R-1608J -> my_rcl:R-1608
- R14: value D6 -> 1k; device my_rcl:R-1608J -> my_rcl:R-1608
- R15: value D8 -> 1k; device my_rcl:R-1608J -> my_rcl:R-1608
- R16: value D10 -> 1k; device my_rcl:R-1608J -> my_rcl:R-1608
- R17: value D12 -> 1k; device my_rcl:R-1608J -> my_rcl:R-1608
- R19: value D3 -> 1k; device my_rcl:R-1608J -> my_rcl:R-1608
Connections:
- removed net +1V0CORE: C12.1, C14.1, C17.1, C9.1, IC4G$1.VCC, IC4G$1.VCCECLK, J8.2, TP3.1
- removed net +5V: C1.1, C2.1, FB3.1, IC1.IN
- removed net +5VD: SW1.1, U1.+5VD
- removed net ADC_D0: IC4G$8.PL24B, R11.2
- removed net ADC_D1: IC4G$8.PL24A, R18.1
- removed net ADC_D10: IC4G$8.PL26A, R16.2
- removed net ADC_D11: IC4G$8.PL26B, R23.1
- removed net ADC_D12: IC4G$8.PL38A, R17.2
- removed net ADC_D13: IC4G$8.PL38B, R24.1
- removed net ADC_D2: IC4G$8.PL30B, R12.2
- removed net ADC_D3: IC4G$8.PL30A, R19.1
- removed net ADC_D4: IC4G$8.PL32A, R13.2
- removed net ADC_D5: IC4G$8.PL32B, R20.1
- removed net ADC_D6: IC4G$8.PL36A, R14.2
- removed net ADC_D7: IC4G$8.PL36B, R21.1
- removed net ADC_D8: IC4G$8.PL42A, R15.2
- removed net ADC_D9: IC4G$8.PL42B, R22.1
- removed net CLK_20M: IC4G$3.PR19A, R1.2
- removed net FT_+5V: F1.P$2, SW1.3, TP21.1
- removed net FT_RD: IC4G$4.PR27B, R35.2
- removed net FT_WR: IC4G$4.PR38A, R34.2
- removed net HV_IO0: IC4G$9.PL8A, JP4.3
- removed net HV_IO1: IC4G$9.PL3A, JP4.4
- removed net HV_IO2: IC4G$9.PL8B, JP4.5
- removed net HV_IO3: IC4G$9.PL3B, JP4.6
- removed net LED3: D4.A, IC4G$3.PR13B
- removed net LV_IO0: IC4G$7.PB4A, JP3.3
- removed net LV_IO1: IC4G$7.PB6A, JP3.4
- removed net LV_IO10: IC4G$6.PB18A, JP3.13
- removed net LV_IO11: IC4G$6.PB18B, JP3.14
- removed net LV_IO12: IC4G$6.PB22A, JP3.15
- removed net LV_IO13: IC4G$6.PB22B, JP3.16
- removed net LV_IO14: IC4G$6.PB24A, JP3.17
- removed net LV_IO15: IC4G$6.PB24B, JP3.18
- removed net LV_IO16: IC4G$5.PB62B, JP3.23
- removed net LV_IO17: IC4G$5.PB54A, JP3.24
- removed net LV_IO18: IC4G$5.PB54B, JP3.25
- removed net LV_IO19: IC4G$5.PB58A, JP3.26
- removed net LV_IO2: IC4G$7.PB4B, JP3.5
- removed net LV_IO20: IC4G$5.PB58B, JP3.27
- removed net LV_IO21: IC4G$5.PB60A, JP3.28
- removed net LV_IO22: IC4G$5.PB60B, JP3.29
- removed net LV_IO23: IC4G$5.PB72A, JP3.30
- removed net LV_IO24: IC4G$5.PB72B, JP3.31
- removed net LV_IO25: IC4G$5.PB74A, JP3.32
- removed net LV_IO26: IC4G$5.PB80A, JP3.33
- removed net LV_IO27: IC4G$5.PB74B, JP3.34
- removed net LV_IO28: IC4G$5.PB76A, JP3.35
- removed net LV_IO29: IC4G$5.PB76B, JP3.36
- removed net LV_IO3: IC4G$7.PB10A, JP3.6
- removed net LV_IO30: IC4G$5.PB78B, JP3.37
- removed net LV_IO31: IC4G$5.PB78A, JP3.38
- removed net LV_IO4: IC4G$7.PB8A, JP3.7
- removed net LV_IO5: IC4G$7.PB10B, JP3.8
- removed net LV_IO6: IC4G$7.PB8B, JP3.9
- removed net LV_IO7: IC4G$7.PB12A, JP3.10
- removed net LV_IO8: IC4G$7.PB6B, JP3.11
- removed net LV_IO9: IC4G$7.PB12B, JP3.12
- removed net N$17: IC6.AD3, R28.2
- removed net N$18: IC6.AD4, R29.2
- removed net N$19: IC6.AD5, R30.2
- removed net N$20: FB1.1, U1.V+
- removed net N$21: FB2.2, U1.V-
- removed net N$5: D4.K, R41.2
- removed net N$6: TP20.1, U1.VIN-
- removed net N$61: CON1.31, R17.1
- removed net N$62: CON1.27, R16.1
- removed net N$63: CON1.23, R15.1
- removed net N$64: CON1.19, R14.1
- removed net N$65: CON1.15, R13.1
- removed net N$66: CON1.11, R12.1
- removed net N$67: CON1.7, R11.1
- removed net N$68: CON1.10, R18.2
- removed net N$69: CON1.14, R19.2
- removed net N$7: TP19.1, U1.VIN+
- removed net N$70: CON1.18, R20.2
- removed net N$71: CON1.22, R21.2
- removed net N$72: CON1.26, R22.2
- removed net N$73: CON1.30, R23.2
- removed net N$74: CON1.34, R24.2
- removed net N$75: IC6.AD6, R31.2
- removed net N$76: IC6.AD7, R32.2
- removed net N$77: IC6.AC2, R35.1
- removed net N$78: F1.P$1, IC6.5V0
- removed net N$8: R1.1, X1.OUT
- removed net UART_TX: IC4G$9.PL4B, TP23.1
- removed net V+: C31.1, CON1.3, CON1.4, FB1.2
- removed net V-: C32.2, CON1.1, CON1.2, FB2.1
- removed net VCCIO2: C20.1, C25.1, IC4G$4.VCCIO2, J4.2, TP6.1
- removed net VCCIO3: C22.1, C26.1, IC4G$5.VCCIO3, J6.2, TP8.1
- removed net VCCIO4: C23.1, C28.1, IC4G$6.VCCIO4, IC4G$7.VCCIO5, J7.2, JP3.19, JP3.22, TP9.1
- removed net VCCIO6: C21.1, C29.1, C30.1, IC4G$8.VCCIO6, IC4G$9.VCCIO7, J5.2, TP7.1
- new net DRAM_+1V8: C36.1, FB2.1, IC8.VCC, IC8.VCCQ
- new net DRAM_CKN: IC4G$6.PB28A, IC8.!CK
- new net DRAM_CKP: IC4G$6.PB28B, IC8.CK
- new net DRAM_CS: IC4G$6.PB26A, IC8.!CS
- new net DRAM_DQ0: IC4G$6.PB22A, IC8.DQ0
- new net DRAM_DQ1: IC4G$6.PB30B, IC8.DQ1
- new net DRAM_DQ2: IC4G$6.PB18B, IC8.DQ2
- new net DRAM_DQ3: IC4G$6.PB18A, IC8.DQ3
- new net DRAM_DQ4: IC4G$6.PB16B, IC8.DQ4
- new net DRAM_DQ5: IC4G$6.PB22B, IC8.DQ5
- new net DRAM_DQ6: IC4G$6.PB24B, IC8.DQ6
- new net DRAM_DQ7: IC4G$6.PB24A, IC8.DQ7
- new net DRAM_NRST: IC4G$6.PB20B, IC8.!RESET
- new net DRAM_RWDS: IC4G$6.PB30A, IC8.RWDS
- new net FT_+1V8: C33.1, IC7.VCORE1, IC7.VCORE2, IC7.VREGOUT
- new net FT_+3V3: C30.1, FB1.2, IC6.VCC, IC7.VCCIO1, IC7.VCCIO2, IC7.VCCIO3, IC7.VPHY, IC7.VPLL, IC7.VREGIN, R11.1, R14.1
- new net FT_NOE: IC4G$9.PL10B, IC7.ACBUS6
- new net FT_NRD: IC4G$9.PL4A, IC7.ACBUS2
- new net FT_NWR: IC4G$9.PL6B, IC7.ACBUS3
- new net FT_SIWU: IC4G$9.PL19A, IC7.ACBUS4
- new net IOH0: CON2.50, IC4G$4.PR24B
- new net IOH1: CON2.48, IC4G$4.PR27A
- new net IOH10: CON2.39, IC4G$4.PR27B
- new net IOH100: CON3.18, IC4G$8.PL44B
- new net IOH101: CON3.20, IC4G$8.PL44A
- new net IOH102: CON3.22, IC4G$8.PL38B
- new net IOH103: CON3.24, IC4G$8.PL38A
- new net IOH104: CON3.26, IC4G$8.PL26B
- new net IOH105: CON3.28, IC4G$8.PL26A
- new net IOH106: CON3.17, IC4G$8.PL42B
- new net IOH107: CON3.19, IC4G$8.PL42A
- new net IOH108: CON3.21, IC4G$8.PL36B
- new net IOH109: CON3.23, IC4G$8.PL36A
- new net IOH11: CON2.37, IC4G$4.PR32B
- new net IOH110: CON3.25, IC4G$8.PL32B
- new net IOH111: CON3.27, IC4G$8.PL32A
- new net IOH112: CON3.29, IC4G$8.PL30A
- new net IOH113: CON3.31, IC4G$8.PL30B
- new net IOH114: CON3.30, IC4G$8.PL24A
- new net IOH115: CON3.32, IC4G$8.PL24B
- new net IOH12: CON2.35, IC4G$4.PR42A
- new net IOH13: CON2.33, IC4G$4.PR42B
- new net IOH14: CON2.47, IC4G$4.PR26A
- new net IOH15: CON2.51, IC4G$3.PR13B
- new net IOH16: CON2.49, IC4G$3.PR17A
- new net IOH17: CON2.40, IC4G$4.PR34A
- new net IOH18: CON2.42, IC4G$4.PR36B
- new net IOH2: CON2.46, IC4G$4.PR24A
- new net IOH3: CON2.44, IC4G$4.PR36A
- new net IOH4: CON2.38, IC4G$4.PR34B
- new net IOH5: CON2.36, IC4G$4.PR38B
- new net IOH6: CON2.34, IC4G$4.PR38A
- new net IOH7: CON2.45, IC4G$4.PR30A
- new net IOH8: CON2.43, IC4G$4.PR32A
- new net IOH9: CON2.41, IC4G$4.PR30B
- new net IOL0: CON2.26, IC4G$5.PB84A
- new net IOL1: CON2.24, IC4G$5.PB84B
- new net IOL10: CON2.6, IC4G$5.PB74B
- new net IOL101: CON3.4, IC4G$7.PB12B
- new net IOL102: CON3.6, IC4G$7.PB12A
- new net IOL103: CON3.8, IC4G$7.PB8B
- new net IOL104: CON3.3, IC4G$7.PB10B
- new net IOL105: CON3.5, IC4G$7.PB8A
- new net IOL106: CON3.7, IC4G$7.PB10A
- new net IOL107: CON3.9, IC4G$7.PB4B
- new net IOL108: CON3.10, IC4G$7.PB6B
- new net IOL109: CON3.12, IC4G$7.PB6A
- new net IOL11: CON2.29, IC4G$5.PB66A
- new net IOL110: CON3.11, IC4G$8.PL47A
- new net IOL111: CON3.13, IC4G$7.PB4A
- new net IOL12: CON2.27, IC4G$5.PB66B
- new net IOL13: CON2.25, IC4G$5.PB70A
- new net IOL14: CON2.23, IC4G$5.PB70B
- new net IOL15: CON2.21, IC4G$5.PB64B
- new net IOL16: CON2.19, IC4G$5.PB68B
- new net IOL17: CON2.17, IC4G$5.PB64A
- new net IOL18: CON2.15, IC4G$5.PB68A
- new net IOL19: CON2.13, IC4G$5.PB72B
- new net IOL2: CON2.22, IC4G$5.PB82B
- new net IOL20: CON2.4, IC4G$5.PB74A
- new net IOL21: CON2.11, IC4G$5.PB72A
- new net IOL22: CON2.9, IC4G$5.PB60B
- new net IOL23: CON2.7, IC4G$5.PB60A
- new net IOL24: CON2.5, IC4G$5.PB58B
- new net IOL25: CON2.3, IC4G$5.PB58A
- new net IOL3: CON2.20, IC4G$5.PB82A
- new net IOL4: CON2.18, IC4G$5.PB80B
- new net IOL5: CON2.16, IC4G$5.PB80A
- new net IOL6: CON2.14, IC4G$5.PB78A
- new net IOL7: CON2.12, IC4G$5.PB78B
- new net IOL8: CON2.10, IC4G$5.PB76B
- new net IOL9: CON2.8, IC4G$5.PB76A
- new net USB_+5V: CON1.VBUS
- new net USB_DM: CON1.D-, IC7.DM
- new net USB_DP: CON1.D+, IC7.DP
- net +1V0: now also C12.1, C14.1, C8.1, IC4G$1.VCC, IC4G$1.VCCECLK; no longer J8.1
- net +1V8: now also C10.1, C26.1, C28.1, C29.1, FB2.2, IC4G$5.VCCIO3, IC4G$6.VCCIO4, IC4G$7.VCCIO5; no longer C11.1, C18.1, J6.1, J7.1, JP3.2, JP3.39, TP4.1
- net +3V3: now also C11.1, C24.1, C25.1, C34.1, C35.1, FB1.1, IC4G$2.VCCIO0, IC4G$3.VCCIO1, IC4G$4.VCCIO2, IC4G$8.VCCIO6, IC4G$9.VCCIO7, R10.2, R2.2, R3.2, R5.2, R6.2, R7.2, R8.2, R9.2; no longer C5.1, IC1.OUT, J3.1, J4.1, J5.1, JP4.2
- net ADC_DN1: now also CON2.30; no longer TP2.1
- net ADC_DP1: now also CON2.28; no longer TP1.1
- net DONE: no longer JP2.6
- net FLASH_CS: no longer JP2.1
- net FLASH_MISO: no longer JP2.2
- net FLASH_MOSI: no longer JP2.5
- net FLASH_SCK: no longer JP2.3
- net FT_CLK: now also IC4G$9.PL10A, IC7.ACBUS5; no longer IC4G$4.PR32A, R33.2
- net FT_D0: now also IC4G$9.PL17B, IC7.ADBUS0; no longer IC4G$4.PR24B, R25.1
- net FT_D1: now also IC4G$9.PL11A, IC7.ADBUS1; no longer IC4G$4.PR27A, R26.1
- net FT_D2: now also IC4G$9.PL11B, IC7.ADBUS2; no longer IC4G$4.PR24A, R27.1
- net FT_D3: now also IC4G$9.PL17A, IC7.ADBUS3; no longer IC4G$4.PR36A, R28.1
- net FT_D4: now also IC4G$9.PL3B, IC7.ADBUS4; no longer IC4G$4.PR36B, R29.1
- net FT_D5: now also IC4G$9.PL8B, IC7.ADBUS5; no longer IC4G$4.PR34A, R30.1
- net FT_D6: now also IC4G$9.PL3A, IC7.ADBUS6; no longer IC4G$4.PR34B, R31.1
- net FT_D7: now also IC4G$9.PL8A, IC7.ADBUS7; no longer IC4G$4.PR38B, R32.1
- net FT_RXNF: now also IC4G$9.PL4B, IC7.ACBUS0; no longer IC4G$4.PR32B, R37.2
- net FT_TXNE: now also IC4G$9.PL6A, IC7.ACBUS1; no longer IC4G$4.PR42B, R36.2
- net GND: now also C32.2, C33.2, C34.2, C35.2, C36.2, CON1.GND, CON1.XT, CON2.1, CON2.2, CON2.31, CON2.32, CON3.1, CON3.14, CON3.15, CON3.16, CON3.2, IC6.VSS, IC7.GND1, IC7.GND2, IC7.GND3, IC7.HT, IC7.TEST, IC8.VSS, IC8.VSSQ, R13.2, R15.1, R16.1, R17.1, R19.1, X2.GND; no longer C1.2, C17.2, C18.2, C19.2, C2.2, C20.2, C21.2, C22.2, C23.2, C32.1, C5.2, C9.2, CON1.12, CON1.13, CON1.16, CON1.17, CON1.20, CON1.21, CON1.24, CON1.25, CON1.28, CON1.29, CON1.32, CON1.33, CON1.5, CON1.6, CON1.8, CON1.9, IC1.GND, IC6.GND1, IC6.GND2, JP1.4, JP2.4, JP3.1, JP3.20, JP3.21, JP3.40, JP4.1, R38.1, R39.1, R40.1, R41.1, R42.1, TP10.1, TP11.1, TP12.1, TP13.1, TP14.1, TP15.1, TP16.1, TP17.1, TP18.1, TP22.1, TP24.1, U1.GND1, U1.GND2, X1.GND
- net JTAG_EN: no longer JP1.6
- net JTAG_TCK: now also IC7.BDBUS0; no longer JP1.3
- net JTAG_TDI: now also IC7.BDBUS1; no longer JP1.2
- net JTAG_TDO: now also IC7.BDBUS2; no longer JP1.5
- net JTAG_TMS: now also IC7.BDBUS3; no longer JP1.1
- net LED0: now also IC4G$3.PR20A; no longer IC4G$3.PR20B
- net LED1: now also IC4G$3.PR20B; no longer IC4G$3.PR20A
- net LED2: now also IC4G$3.PR19A; no longer IC4G$3.SCL
- net N$1: now also R19.2; no longer R42.2
- net N$10: now also IC6.DI, IC7.EEDATA; no longer IC6.AC0, R37.1
- net N$11: now also IC6.CS, IC7.EECS, R12.2; no longer IC6.AC1, R36.1
- net N$12: now also IC6.DO, R11.2, R12.1; no longer IC6.AC3, R34.1
- net N$13: now also C32.1, IC7.OSCO, X2.2; no longer IC6.AC5, R33.1
- net N$14: now also C31.1, IC7.OSCI, X2.1; no longer IC6.AD0, R25.2
- net N$15: now also IC7.REF, R13.1; no longer IC6.AD1, R26.2
- net N$16: now also IC7.RESET#, R14.2; no longer IC6.AD2, R27.2
- net N$2: now also R15.2; no longer R38.2
- net N$3: now also R16.2; no longer R39.2
- net N$4: now also R17.2; no longer R40.2
- net N$9: now also IC6.CLK, IC7.EECLK; no longer FB3.2, SW1.2
- net PROGRAMN: no longer JP2.7
- net VCCIO0: no longer C10.1, C19.1, C24.1, C8.1, IC4G$2.VCCIO0, IC4G$3.VCCIO1, J3.2, JP1.7, R10.2, R2.2, R3.2, R5.2, R6.2, R7.2, R8.2, R9.2, TP5.1, X1.EN, X1.VCC
Other:
- note added: "DRAM"
- note added: "USB Interface"
- moved on the sheet: C10, C11, C25, C26, C28, C29, C30, C8, D5, FB1, FB2, R11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

Commit message: 4層DRC
Parts:
- removed C31, C32: 22p, my_rcl:C-1608
- removed C33, C36: 10u, my_rcl:C-1608
- removed C34, C35: 0.1u, my_rcl:C-1608
- removed J1, J2: SJ-1608, my_rcl:SJ-1608
- added C1, C18, C21, C22, C23, C5: 0.1u, my_rcl:C-1608
- added C17, C19, C9: 0.1u, my_rcl:C-1005
- added C2, C20: 10u, my_rcl:C-1608
- added D4: LED2, my_rcl:LED-SMD1608
- added FB3: 1.8V, my_rcl:FB
- added FB4, FB6: FT, my_rcl:FB
- added FB5: DRAM, my_rcl:FB
- added IC1: 3.3V, my_ic:TLV740
- added R1, R18: 1k, my_rcl:R-1608
- C10: value 0.1u -> 10u; device my_rcl:C-1005 -> my_rcl:C-2012
- C11: device my_rcl:C-1608 -> my_rcl:C-1005
- C24, C25: value 0.1u -> 22p; device my_rcl:C-1005 -> my_rcl:C-1608
- C26: value 0.1u -> 10u
- C29, C8: value 0.1u -> 10u; device my_rcl:C-1608 -> my_rcl:C-2012
- C30: value 10u -> 0.1u
- C6: device my_rcl:C-2012 -> my_rcl:C-1608
- CON1: value USB-A -> MEZZANINE_2X30; device my_connector:USB-A -> my_connector:MEZZANINE_2X30
- CON3: value MEZZANINE_2X30 -> USB-SC; device my_connector:MEZZANINE_2X30 -> my_connector:USB-SC
- D1: value LED0 -> USB; device my_rcl:LED-SMD1608 -> my_rcl:SBD-1A2
- D2: value LED1 -> LED0
- D3: value LED2 -> LED1
- FB1: value FB -> 3.3V
- FB2: value FB -> 1.0V
- IC2: value 1.8V -> MPM3804; device my_ic:TLV740 -> my_ic:MPM3804
- R12: value 1k -> 10k
- R13: value 12.1k -> 1k
- R14: value 1k -> 12.1k
- R2: value 10k -> 1k
- renumbered X2 to X1
Connections:
- removed net LDO1V0: C4.1, IC3.EN, IC3.IN, J2.2
- removed net LDO1V8: C3.1, IC2.EN, IC2.IN, J1.2
- removed net N$2 (its old number): D1.K, R15.2
- removed net VCCIO0: C27.1, IC5.HOLD, IC5.VCC, IC5.WP
- new net +1V0_LDO: C5.1, FB2.1, IC3.OUT
- new net +1V8_DCDC: C6.1, FB3.1, IC2.OUT, R1.2
- new net +3.3V_LDO: C4.1, FB1.1, IC1.OUT
- new net N$4: D4.K, R18.2
- new net N$7: IC2.FB, R1.1, R2.2
- new net VIN: C1.1, C2.1, CON2.57, CON2.58, CON2.59, CON2.60, D1.K, IC1.EN, IC1.IN, IC2.EN, IC2.VIN
- net +1V0: now also C9.1, FB2.2; no longer C7.1, IC3.OUT
- net +1V8: now also C11.1, C19.1, C3.1, CON1.55, CON1.56, CON2.45, CON2.46, CON2.47, CON2.48, FB3.2, FB5.2, FB6.1, IC3.EN, IC3.IN; no longer C16.1, C26.1, C28.1, C29.1, C6.1, FB2.2, IC2.OUT
- net +3V3: now also C16.1, C17.1, C18.1, C7.1, CON1.59, CON1.60, CON2.49, CON2.50, CON2.51, CON2.52, FB1.2, FB4.1, IC5.HOLD, IC5.VCC, IC5.WP, R11.2, R4.2; no longer C11.1, C24.1, C25.1, C34.1, C35.1, FB1.1, J1.1, J2.1, R2.2, R5.2
- net ADC_DN1: now also CON1.30; no longer CON2.30
- net ADC_DP1: now also CON1.28; no longer CON2.28
- net DONE: now also R10.1; no longer R9.1
- net DRAM_+1V8: now also C29.1, C30.1, FB5.1; no longer C36.1, FB2.1
- net FLASH_CS: now also R11.1; no longer R10.1
- net FT_+1V8: now also C26.1, C27.1, C28.1, FB6.2; no longer C33.1, IC7.VREGOUT
- net FT_+3V3: now also C20.1, C21.1, C22.1, C23.1, FB4.2, R12.1, R15.1; no longer C30.1, FB1.2, IC7.VREGIN, R11.1, R14.1
- net GND: now also C1.2, C17.2, C18.2, C19.2, C2.2, C20.2, C21.2, C22.2, C23.2, C5.2, C9.2, CON1.1, CON1.2, CON1.31, CON1.32, CON1.52, CON1.53, CON1.54, CON1.57, CON1.58, CON2.14, CON2.15, CON2.16, CON2.33, CON2.34, CON2.35, CON2.36, CON2.37, CON2.38, CON2.39, CON2.40, CON2.41, CON2.42, CON2.43, CON2.44, CON2.53, CON2.54, CON2.55, CON2.56, CON3.GND, CON3.XT, IC1.GND, R14.2, R18.1, R2.1, R5.1; no longer C31.2, C32.2, C33.2, C34.2, C35.2, C36.2, CON1.GND, CON1.XT, CON2.31, CON2.32, CON3.1, CON3.14, CON3.15, CON3.16, CON3.2, R13.2, R15.1, R4.1
- net INITN: now also R8.1; no longer R7.1
- net IOH0: now also CON1.50; no longer CON2.50
- net IOH1: now also CON1.48; no longer CON2.48
- net IOH10: now also CON1.39; no longer CON2.39
- net IOH100: now also CON2.18; no longer CON3.18
- net IOH101: now also CON2.20; no longer CON3.20
- net IOH102: now also CON2.22; no longer CON3.22
- net IOH103: now also CON2.24; no longer CON3.24
- net IOH104: now also CON2.26; no longer CON3.26
- net IOH105: now also CON2.28; no longer CON3.28
- net IOH106: now also CON2.17; no longer CON3.17
- net IOH107: now also CON2.19; no longer CON3.19
- net IOH108: now also CON2.21; no longer CON3.21
- net IOH109: now also CON2.23; no longer CON3.23
- net IOH11: now also CON1.37; no longer CON2.37
- net IOH110: now also CON2.25; no longer CON3.25
- net IOH111: now also CON2.27; no longer CON3.27
- net IOH112: now also CON2.29; no longer CON3.29
- net IOH113: now also CON2.31; no longer CON3.31
- net IOH114: now also CON2.30; no longer CON3.30
- net IOH115: now also CON2.32; no longer CON3.32
- net IOH12: now also CON1.35; no longer CON2.35
- net IOH13: now also CON1.33; no longer CON2.33
- net IOH14: now also CON1.47; no longer CON2.47
- net IOH15: now also CON1.51; no longer CON2.51
- net IOH16: now also CON1.49; no longer CON2.49
- net IOH17: now also CON1.40; no longer CON2.40
- net IOH18: now also CON1.42; no longer CON2.42
- net IOH2: now also CON1.46; no longer CON2.46
- net IOH3: now also CON1.44; no longer CON2.44
- net IOH4: now also CON1.38; no longer CON2.38
- net IOH5: now also CON1.36; no longer CON2.36
- net IOH6: now also CON1.34; no longer CON2.34
- net IOH7: now also CON1.45; no longer CON2.45
- net IOH8: now also CON1.43; no longer CON2.43
- net IOH9: now also CON1.41; no longer CON2.41
- net IOL0: now also CON1.26; no longer CON2.26
- net IOL1: now also CON1.24; no longer CON2.24
- net IOL10: now also CON1.6; no longer CON2.6
- net IOL101: now also CON2.4; no longer CON3.4
- net IOL102: now also CON2.6; no longer CON3.6
- net IOL103: now also CON2.8; no longer CON3.8
- net IOL104: now also CON2.3; no longer CON3.3
- net IOL105: now also CON2.5; no longer CON3.5
- net IOL106: now also CON2.7; no longer CON3.7
- net IOL107: now also CON2.9; no longer CON3.9
- net IOL108: now also CON2.10; no longer CON3.10
- net IOL109: now also CON2.12; no longer CON3.12
- net IOL11: now also CON1.29; no longer CON2.29
- net IOL110: now also CON2.11; no longer CON3.11
- net IOL111: now also CON2.13; no longer CON3.13
- net IOL12: now also CON1.27; no longer CON2.27
- net IOL13: now also CON1.25; no longer CON2.25
- net IOL14: now also CON1.23; no longer CON2.23
- net IOL15: now also CON1.21; no longer CON2.21
- net IOL16: now also CON1.19; no longer CON2.19
- net IOL17: now also CON1.17; no longer CON2.17
- net IOL18: now also CON1.15; no longer CON2.15
- net IOL19: now also CON1.13; no longer CON2.13
- net IOL2: now also CON1.22; no longer CON2.22
- net IOL20: now also CON1.4; no longer CON2.4
- net IOL21: now also CON1.11; no longer CON2.11
- net IOL22: now also CON1.9; no longer CON2.9
- net IOL23: now also CON1.7; no longer CON2.7
- net IOL24: now also CON1.5; no longer CON2.5
- net IOL25: now also CON1.3; no longer CON2.3
- net IOL3: now also CON1.20; no longer CON2.20
- net IOL4: now also CON1.18; no longer CON2.18
- net IOL5: now also CON1.16; no longer CON2.16
- net IOL6: now also CON1.14; no longer CON2.14
- net IOL7: now also CON1.12; no longer CON2.12
- net IOL8: now also CON1.10; no longer CON2.10
- net IOL9: now also CON1.8; no longer CON2.8
- net JTAG_EN: now also R7.1; no longer R6.1
- net JTAG_TCK: now also R5.2; no longer R4.2
- net JTAG_TDI: now also R4.1; no longer R3.1
- net JTAG_TDO: now also R3.1; no longer R2.1
- net JTAG_TMS: now also R6.1; no longer R5.1
- net LED0: now also D2.A; no longer D1.A
- net LED1: now also D3.A; no longer D2.A
- net LED2: now also D4.A; no longer D3.A
- net N$11: now also R13.2; no longer R12.2
- net N$12: now also R12.2, R13.1; no longer R11.2, R12.1
- net N$13: now also C25.1; no longer C32.1
- net N$14: now also C24.1; no longer C31.1
- net N$15: now also R14.1; no longer R13.1
- net N$16: now also R15.2; no longer R14.2
- net PROGRAMN: now also R9.1; no longer R8.1
- net USB_+5V: now also CON3.VBUS, D1.A; no longer CON1.VBUS
- net USB_DM: now also CON3.D-; no longer CON1.D-
- net USB_DP: now also CON3.D+; no longer CON1.D+
Other:
- moved on the sheet: C10, C11, C16, C24, C25, C26, C27, C28, C29, C3, C30, C4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

Commit message: 6層
Parts:
- added C31, C32: 10u, my_rcl:C-1608
- added C33, C34: 0.1u, my_rcl:C-1608
- added FB7: VIN, my_rcl:FB
- C4, C5: value 0.1u -> 1u
- R1: value 1k -> 10k
- R2: value 1k -> 5k
Connections:
- new net 1.8V_DCDC_SW: IC2.SW
- new net VIN_DCDC: C1.1, C2.1, C31.1, C32.1, FB7.2, IC1.EN, IC1.IN, IC2.EN, IC2.VIN
- net DRAM_+1V8: now also C33.1
- net GND: now also C31.2, C32.2, C33.2, C34.2
- net VIN: now also C34.1, FB7.1; no longer C1.1, C2.1, IC1.EN, IC1.IN, IC2.EN, IC2.VIN
Other:
- moved on the sheet: C29, C30, D1, FB5

Commit message: 発注
Parts:
- added C35: 0.1u, my_rcl:C-1608
- added J1: CLK, my_rcl:SJ-1608
- added X2: 12MHz, my_rcl:CRYSTAL2
- C11, C13: value 0.1u -> 10u; device my_rcl:C-1005 -> my_rcl:C-2012
- C18, C21, C23: device my_rcl:C-1608 -> my_rcl:C-1005
- C19: device my_rcl:C-1005 -> my_rcl:C-1608
- C20: value 10u -> 0.1u; device my_rcl:C-1608 -> my_rcl:C-1005
- C24: value 22p -> 10u
- C25: value 22p -> 0.1u
- C26, C31, C32, C6: value 10u -> 0.1u
- C28: value 0.1u -> 22p
- C29: value 10u -> 22p; device my_rcl:C-2012 -> my_rcl:C-1608
- C3, C30: value 0.1u -> 10u
- C34: value 0.1u -> 10u; device my_rcl:C-1608 -> my_rcl:C-2012
- C4: value 1u -> 0.1u
- C5: value 1u -> 10u
- C7, C8: value 10u -> 1u; device my_rcl:C-2012 -> my_rcl:C-1608
- C9: value 0.1u -> 10u; device my_rcl:C-1005 -> my_rcl:C-1608
- FB1: value 3.3V -> VIN
- FB2: value 1.0V -> 3.3V
- FB3: value 1.8V -> 1.0V
- FB4: value FT -> 1.8V
- FB5: value DRAM -> FT
- FB7: value VIN -> DRAM
- IC8: value HYPERRAM -> HyperRAM
- X1: value 12MHz -> 25MHz; device my_rcl:CRYSTAL2 -> my_rcl:OSC-KC3225
Connections:
- new net N$6: J1.1, X1.OUT
- net +1V0: now also C11.1, C15.1, C17.1, FB3.2; no longer C14.1, C8.1, C9.1, FB2.2
- net +1V0_LDO: now also C8.1, FB3.1; no longer C5.1, FB2.1
- net +1V8: now also C14.1, C16.1, C18.1, C23.1, C6.1, FB4.2, FB7.2; no longer C10.1, C11.1, C15.1, C19.1, C3.1, FB3.2, FB5.2
- net +1V8_DCDC: now also C9.1, FB4.1; no longer C6.1, FB3.1
- net +3.3V_LDO: now also C7.1, FB2.1; no longer C4.1, FB1.1
- net +3V3: now also C10.1, C19.1, C20.1, C21.1, C22.1, FB2.2, FB5.1, X1.EN, X1.VCC; no longer C16.1, C17.1, C18.1, C7.1, FB1.2, FB4.1
- net DRAM_+1V8: now also C34.1, C35.1, FB7.1; no longer C29.1, C30.1, FB5.1
- net FT_+1V8: now also C30.1, C31.1, C32.1; no longer C26.1, C27.1, C28.1
- net FT_+3V3: now also C24.1, C25.1, C26.1, C27.1, FB5.2; no longer C20.1, C21.1, C22.1, C23.1, FB4.2
- net GND: now also C35.2, X2.GND
- net IOH112: now also J1.2
- net N$13: now also C29.1, X2.2; no longer C25.1, X1.2
- net N$14: now also C28.1, X2.1; no longer C24.1, X1.1
- net VIN: now also C1.1, FB1.1; no longer C34.1, FB7.1
- net VIN_DCDC: now also C3.1, C4.1, C5.1, FB1.2; no longer C1.1, C31.1, C32.1, FB7.2
Other:
- moved on the sheet: C1, C10, C11, C12, C13, C14, C15, C16, C17, C18, C19, C2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
