File: ADC3_FPGA_BGA.sch (EAGLE design)
At the start: 80 parts, among them CON1 MEZZANINE_2X30, CON2 MEZZANINE_2X30, CON3 USB-SC, IC1 3.3V, IC2 MPM3804, IC3 1.0V, IC4 LFD2NX-40, IC5 EEPROM, IC6 93LC56, IC7 FT2232H, IC8 HyperRAM, J1 CLK, X1 25MHz, X2 12MHz

Commit message: Artix-7 途中
Parts:
- removed X2: 12MHz, my_rcl:CRYSTAL2
- added C36, C37, C38: 1u, my_rcl:C-1005
- added C39, C41, C42, C43, C47, C48, C49, C51: 0.1u, my_rcl:C-1608
- added C40, C46: 10u, my_rcl:C-1608
- added C44, C45: 22p, my_rcl:C-1608
- added C50: 10u, my_rcl:C-2012
- added D6: PWR, my_rcl:LED-SMD1608
- added FB8: DRAM, my_rcl:FB
- added IC9: HyperRAM, my_ic:HYPERRAM
- added J2: BANK35, my_rcl:SJ-3
- added R20: 1k, my_rcl:R-1608
- added TP1: TMS, my_connector:TESTPIN-PAD
- added TP2: TDI, my_connector:TESTPIN-PAD
- added TP3: TCK, my_connector:TESTPIN-PAD
- added TP4: TDO, my_connector:TESTPIN-PAD
- added TP5: GND, my_connector:TESTPIN-PAD
- C10, C11, C13, C34: value 10u -> 1u; device my_rcl:C-2012 -> my_rcl:C-1005
- C12, C14, C15: value 0.1u -> 1u
- C16, C17, C18: value 0.1u -> 10u; device my_rcl:C-1005 -> my_rcl:C-1608
- C19, C4: value 0.1u -> 10u
- C2, C24: device my_rcl:C-1608 -> my_rcl:C-2012
- C20, C21, C23: value 0.1u -> 10u; device my_rcl:C-1005 -> my_rcl:C-2012
- C22, C25: value 0.1u -> 10u; device my_rcl:C-1608 -> my_rcl:C-2012
- C26, C27, C31, C32, C33, C35: value 0.1u -> 1u; device my_rcl:C-1608 -> my_rcl:C-1005
- C28, C29: value 22p -> 1u; device my_rcl:C-1608 -> my_rcl:C-1005
- C30, C9: value 10u -> 1u; device my_rcl:C-1608 -> my_rcl:C-1005
- C5: value 10u -> 0.1u
- C7, C8: device my_rcl:C-1608 -> my_rcl:C-1005
- D5: value PWR -> LED2
- FB3, IC3: value 1.0V -> 2.5V
- FB5: value FT -> 1.0V
- FB7: value DRAM -> FT
- IC1: value 3.3V -> ARTIX7-FTG256; device my_ic:TLV740 -> my_ic:ARTIX7-FTG256
- IC2: value MPM3804 -> 3.3V; device my_ic:MPM3804 -> my_ic:TLV740
- IC4: value LFD2NX-40 -> MPM3804; device my_ic:LFD2NX-40 -> my_ic:MPM3804
- IC5: value EEPROM -> MPM3804; device my_ic:EEPROM_SPI -> my_ic:MPM3804
- IC6: value 93LC56 -> EEPROM; device my_ic:93LC56 -> my_ic:EEPROM_SPI-WIDE
- IC7: value FT2232H -> 93LC56; device my_ic:FT2232H -> my_ic:93LC56
- IC8: value HyperRAM -> FT2232H-2; device my_ic:HYPERRAM -> my_ic:FT2232H-2
- J1: value CLK -> BANK34; device my_rcl:SJ-1608 -> my_rcl:SJ-3
- R12, R3: value 10k -> 1k
- R13: value 1k -> 12.1k
- R14: value 12.1k -> 1k
- R4: value 10k -> 1.5k
- X1: value 25MHz -> 12MHz; device my_rcl:OSC-KC3225 -> my_rcl:CRYSTAL2
Connections:
- removed net +1V0_LDO: C8.1, FB3.1, IC3.OUT
- removed net +3.3V_LDO: C7.1, FB2.1, IC1.OUT
- removed net ADC_DN1: CON1.30, IC4G$10.ADC_DN1
- removed net ADC_DP1: CON1.28, IC4G$10.ADC_DP1
- removed net INITN: IC4G$2.INITN, R8.1
- removed net JTAG_EN: IC4G$3.JTAG_EN, R7.1
- removed net N$6: J1.1, X1.OUT
- removed net N$7: IC2.FB, R1.1, R2.2
- removed net PB10A: CON2.7, IC4G$7.PB10A
- removed net PB10B: CON2.3, IC4G$7.PB10B
- removed net PB12A: CON2.6, IC4G$7.PB12A
- removed net PB12B: CON2.4, IC4G$7.PB12B
- removed net PB4A: CON2.13, IC4G$7.PB4A
- removed net PB4B: CON2.9, IC4G$7.PB4B
- removed net PB58A: CON1.3, IC4G$5.PB58A
- removed net PB58B: CON1.5, IC4G$5.PB58B
- removed net PB60A: CON1.7, IC4G$5.PB60A
- removed net PB60B: CON1.9, IC4G$5.PB60B
- removed net PB64A: CON1.17, IC4G$5.PB64A
- removed net PB64B: CON1.21, IC4G$5.PB64B
- removed net PB66A: CON1.29, IC4G$5.PB66A
- removed net PB66B: CON1.27, IC4G$5.PB66B
- removed net PB68A: CON1.15, IC4G$5.PB68A
- removed net PB68B: CON1.19, IC4G$5.PB68B
- removed net PB6A: CON2.12, IC4G$7.PB6A
- removed net PB6B: CON2.10, IC4G$7.PB6B
- removed net PB70A: CON1.25, IC4G$5.PB70A
- removed net PB70B: CON1.23, IC4G$5.PB70B
- removed net PB72A: CON1.11, IC4G$5.PB72A
- removed net PB72B: CON1.13, IC4G$5.PB72B
- removed net PB74A: CON1.4, IC4G$5.PB74A
- removed net PB74B: CON1.6, IC4G$5.PB74B
- removed net PB76A: CON1.8, IC4G$5.PB76A
- removed net PB76B: CON1.10, IC4G$5.PB76B
- removed net PB78A: CON1.14, IC4G$5.PB78A
- removed net PB78B: CON1.12, IC4G$5.PB78B
- removed net PB80A: CON1.16, IC4G$5.PB80A
- removed net PB80B: CON1.18, IC4G$5.PB80B
- removed net PB82A: CON1.20, IC4G$5.PB82A
- removed net PB82B: CON1.22, IC4G$5.PB82B
- removed net PB84A: CON1.26, IC4G$5.PB84A
- removed net PB84B: CON1.24, IC4G$5.PB84B
- removed net PB8A: CON2.5, IC4G$7.PB8A
- removed net PB8B: CON2.8, IC4G$7.PB8B
- removed net PL24A: CON2.30, IC4G$8.PL24A
- removed net PL24B: CON2.32, IC4G$8.PL24B
- removed net PL26A: CON2.28, IC4G$8.PL26A
- removed net PL26B: CON2.26, IC4G$8.PL26B
- removed net PL30A: CON2.29, IC4G$8.PL30A, J1.2
- removed net PL30B: CON2.31, IC4G$8.PL30B
- removed net PL32A: CON2.27, IC4G$8.PL32A
- removed net PL32B: CON2.25, IC4G$8.PL32B
- removed net PL36A: CON2.23, IC4G$8.PL36A
- removed net PL36B: CON2.21, IC4G$8.PL36B
- removed net PL38A: CON2.24, IC4G$8.PL38A
- removed net PL38B: CON2.22, IC4G$8.PL38B
- removed net PL42A: CON2.19, IC4G$8.PL42A
- removed net PL42B: CON2.17, IC4G$8.PL42B
- removed net PL44A: CON2.20, IC4G$8.PL44A
- removed net PL44B: CON2.18, IC4G$8.PL44B
- removed net PL47A: CON2.11, IC4G$8.PL47A
- removed net PR13B: CON1.51, IC4G$3.PR13B
- removed net PR17A: CON1.49, IC4G$3.PR17A
- removed net PR24A: CON1.46, IC4G$4.PR24A
- removed net PR24B: CON1.50, IC4G$4.PR24B
- removed net PR26A: CON1.47, IC4G$4.PR26A
- removed net PR27A: CON1.48, IC4G$4.PR27A
- removed net PR27B: CON1.39, IC4G$4.PR27B
- removed net PR30A: CON1.45, IC4G$4.PR30A
- removed net PR30B: CON1.41, IC4G$4.PR30B
- removed net PR32A: CON1.43, IC4G$4.PR32A
- removed net PR32B: CON1.37, IC4G$4.PR32B
- removed net PR34A: CON1.40, IC4G$4.PR34A
- removed net PR34B: CON1.38, IC4G$4.PR34B
- removed net PR36A: CON1.44, IC4G$4.PR36A
- removed net PR36B: CON1.42, IC4G$4.PR36B
- removed net PR38A: CON1.34, IC4G$4.PR38A
- removed net PR38B: CON1.36, IC4G$4.PR38B
- removed net PR42A: CON1.35, IC4G$4.PR42A
- removed net PR42B: CON1.33, IC4G$4.PR42B
- removed net PROGRAMN: IC4G$2.PROG, R9.1
- new net +1V0_DCDC: C19.1, FB5.1, IC5.OUT, R3.2
- new net +1V0_DCDC_FB: IC5.FB, R3.1, R4.2
- new net +1V8_DCDC_FB: IC4.FB, R1.1, R2.2
- new net +2V5: C21.1, CON2.49, CON2.50, FB3.2, J1.3, J2.3
- new net +2V5_LDO: C17.1, FB3.1, IC3.OUT
- new net +3V3_LDO: C16.1, FB2.1, IC2.OUT
- new net 1.0V_DCDC_SW: IC5.SW
- new net INIT_B: IC1G$2.INIT_B, R7.1
- new net IO0_14: CON2.26, IC1G$3.IO_0_14
- new net IO10N_15: CON2.7, IC1G$4.IO_L10N_T1_AD11N_15
- new net IO10N_35: CON1.16, IC1G$6.IO_L10N_T1_AD15N_35
- new net IO10P_15: CON2.9, IC1G$4.IO_L10P_T1_AD11P_15
- new net IO10P_35: CON1.18, IC1G$6.IO_L10P_T1_AD15P_35
- new net IO11N_14: CON2.40, IC1G$3.IO_L11N_T1_SRCC_14
- new net IO11P_14: CON2.38, IC1G$3.IO_L11P_T1_SRCC_14
- new net IO12N_14: CON2.32, IC1G$3.IO_L12N_T1_MRCC_14
- new net IO12N_35: CON1.19, IC1G$6.IO_L12N_T1_MRCC_35
- new net IO12P_14: CON2.30, IC1G$3.IO_L12P_T1_MRCC_14
- new net IO12P_35: CON1.21, IC1G$6.IO_L12P_T1_MRCC_35
- new net IO13N_15: CON2.12, IC1G$4.IO_L13N_T2_MRCC_15
- new net IO13P_15: CON2.14, IC1G$4.IO_L13P_T2_MRCC_15
- new net IO14N_35: CON1.23, IC1G$6.IO_L14N_T2_SRCC_35
- new net IO14P_35: CON1.25, IC1G$6.IO_L14P_T2_SRCC_35
- new net IO15N_15: CON2.10, IC1G$4.IO_L15N_T2_DQS_ADV_B_15
- new net IO15N_35: CON1.20, IC1G$6.IO_L15N_T2_DQS_35
- new net IO15P_15: CON2.8, IC1G$4.IO_L15P_T2_DQS_15
- new net IO15P_35: CON1.22, IC1G$6.IO_L15P_T2_DQS_35
- new net IO17N_15: CON2.11, IC1G$4.IO_L17N_T2_A25_15
- new net IO17N_35: CON1.24, IC1G$6.IO_L17N_T2_35
- new net IO17P_15: CON2.13, IC1G$4.IO_L17P_T2_A26_15
- new net IO17P_35: CON1.26, IC1G$6.IO_L17P_T2_35
- new net IO19N_35: CON1.35, IC1G$6.IO_L19N_T3_VREF_35
- new net IO19P_35: CON1.37, IC1G$6.IO_L19P_T3_35
- new net IO20N_35: CON1.28, IC1G$6.IO_L20N_T3_35
- new net IO20P_35: CON1.30, IC1G$6.IO_L20P_T3_35
- new net IO21N_15: CON2.16, IC1G$4.IO_L21N_T3_DQS_A18_15
- new net IO21N_35: CON1.27, IC1G$6.IO_L21N_T3_DQS_35
- new net IO21P_15: CON2.18, IC1G$4.IO_L21P_T3_DQS_15
- new net IO21P_35: CON1.29, IC1G$6.IO_L21P_T3_DQS_35
- new net IO22N_15: CON2.15, IC1G$4.IO_L22N_T3_A16_15
- new net IO22N_35: CON1.32, IC1G$6.IO_L22N_T3_35
- new net IO22P_15: CON2.17, IC1G$4.IO_L22P_T3_A17_15
- new net IO22P_35: CON1.34, IC1G$6.IO_L22P_T3_35
- new net IO23N_15: CON2.21, IC1G$4.IO_L23N_T3_FWE_B_15
- new net IO23N_35: CON1.38, IC1G$6.IO_L23N_T3_35
- new net IO23P_15: CON2.19, IC1G$4.IO_L23P_T3_FOE_B_15
- new net IO23P_35: CON1.36, IC1G$6.IO_L23P_T3_35
- new net IO24N_15: CON2.20, IC1G$4.IO_L24N_T3_RS0_15
- new net IO24N_35: CON1.31, IC1G$6.IO_L24N_T3_35
- new net IO24P_15: CON2.22, IC1G$4.IO_L24P_T3_RS1_15
- new net IO24P_35: CON1.33, IC1G$6.IO_L24P_T3_35
- new net IO2N_14: CON2.27, IC1G$3.IO_L2N_T0_D03_14
- new net IO2N_34: CON1.42, IC1G$5.IO_L2N_T0_34
- new net IO2N_35: CON1.9, IC1G$6.IO_L2N_T0_AD12N_35
- new net IO2P_14: CON2.25, IC1G$3.IO_L2P_T0_D02_14
- new net IO2P_34: CON1.44, IC1G$5.IO_L2P_T0_34
- new net IO2P_35: CON1.7, IC1G$6.IO_L2P_T0_AD12P_35
- new net IO3N_35: CON1.6, IC1G$6.IO_L3N_T0_DQS_AD5N_35
- new net IO3P_35: CON1.4, IC1G$6.IO_L3P_T0_DQS_AD5P_35
- new net IO4N_14: CON2.31, IC1G$3.IO_L4N_T0_D05_14
- new net IO4N_34: CON1.48, IC1G$5.IO_L4N_T0_34
- new net IO4N_35: CON1.11, IC1G$6.IO_L4N_T0_35
- new net IO4P_14: CON2.29, IC1G$3.IO_L4P_T0_D04_14
- new net IO4P_34: CON1.46, IC1G$5.IO_L4P_T0_34
- new net IO4P_35: CON1.13, IC1G$6.IO_L4P_T0_35
- new net IO5N_34: CON1.43, IC1G$5.IO_L5N_T0_34
- new net IO5N_35: CON1.5, IC1G$6.IO_L5N_T0_AD13N_35
- new net IO5P_14: CON2.28, IC1G$3.IO_L5P_T0_D06_14
- new net IO5P_34: CON1.41, IC1G$5.IO_L5P_T0_34
- new net IO5P_35: CON1.3, IC1G$6.IO_L5P_T0_AD13P_35
- new net IO7N_14: CON2.35, IC1G$3.IO_L7N_T1_D10_14
- new net IO7N_34: CON1.50, IC1G$5.IO_L7N_T1_34
- new net IO7N_35: CON1.15, IC1G$6.IO_L7N_T1_AD6N_35
- new net IO7P_14: CON2.33, IC1G$3.IO_L7P_T1_D09_14
- new net IO7P_34: CON1.52, IC1G$5.IO_L7P_T1_34
- new net IO7P_35: CON1.17, IC1G$6.IO_L7P_T1_AD6P_35
- new net IO8N_14: CON2.39, IC1G$3.IO_L8N_T1_D12_14
- new net IO8N_15: CON2.4, IC1G$4.IO_L8N_T1_AD10N_15
- new net IO8N_34: CON1.47, IC1G$5.IO_L8N_T1_34
- new net IO8N_35: CON1.8, IC1G$6.IO_L8N_T1_AD14N_35
- new net IO8P_14: CON2.37, IC1G$3.IO_L8P_T1_D11_14
- new net IO8P_15: CON2.6, IC1G$4.IO_L8P_T1_AD10P_15
- new net IO8P_34: CON1.45, IC1G$5.IO_L8P_T1_34
- new net IO8P_35: CON1.10, IC1G$6.IO_L8P_T1_AD14P_35
- new net IO9N_14: CON2.36, IC1G$3.IO_L9N_T1_DQS_D13_14
- new net IO9N_15: CON2.3, IC1G$4.IO_L9N_T1_DQS_AD3N_15
- new net IO9N_34: CON1.49, IC1G$5.IO_L9N_T1_DQS_34
- new net IO9N_35: CON1.12, IC1G$6.IO_L9N_T1_DQS_AD7N_35
- new net IO9P_14: CON2.34, IC1G$3.IO_L9P_T1_DQS_14
- new net IO9P_15: CON2.5, IC1G$4.IO_L9P_T1_DQS_AD3P_15
- new net IO9P_34: CON1.51, IC1G$5.IO_L9P_T1_DQS_34
- new net IO9P_35: CON1.14, IC1G$6.IO_L9P_T1_DQS_AD7P_35
- new net LED3: D5.A, IC1G$3.IO_L23P_T3_A03_D19_14
- new net N$5: D5.K, R18.2
- new net PROGRAM_B: IC1G$2.PROGRAM_B, R8.1
- new net VCCO34: C24.1, C26.1, C28.1, IC1G$5.VCCO_34, J1.2
- new net VCCO35: C25.1, C27.1, C29.1, C30.1, IC1G$6.VCCO_35, J2.2
- net +1V0: now also C13.1, C23.1, C7.1, C9.1, FB5.2, IC1G$1.VCCDRAM, IC1G$1.VCCINT; no longer C12.1, C17.1, FB3.2, IC4G$1.VCC, IC4G$1.VCCECLK
- net +1V8: now also C10.1, C12.1, C22.1, C31.1, C33.1, C35.1, C8.1, FB7.1, FB8.2, IC1G$1.VCCADC, IC1G$1.VCCAUX, IC1G$4.VCCO15; no longer C13.1, C16.1, C18.1, C23.1, C6.1, FB6.1, FB7.2, IC3.EN, IC3.IN, IC4G$1.VCCAUX, IC4G$1.VCCAUXA, IC4G$1.VCCAUXH3, IC4G$1.VCCAUXH4, IC4G$1.VCCAUXH5, IC4G$10.ADC_REFP0, IC4G$10.ADC_REFP1, IC4G$10.VCCADC18, IC4G$5.VCCIO3, IC4G$6.VCCIO4, IC4G$7.VCCIO5
- net +1V8_DCDC: now also C18.1, IC4.OUT; no longer C9.1, IC2.OUT
- net +3V3: now also C32.1, C34.1, C36.1, C37.1, C38.1, C39.1, D6.A, FB6.1, IC1G$2.CFGBVS, IC1G$2.M0, IC1G$2.VCCO_0, IC1G$3.IO_L3P_T0_DQS_PUDC_B_14, IC1G$3.VCCO_14, IC6.HOLD, IC6.VCC, IC6.WP, J1.1, J2.1, R5.2; no longer C10.1, C19.1, C21.1, C22.1, CON2.49, CON2.50, D5.A, FB5.1, IC4G$2.VCCIO0, IC4G$3.VCCIO1, IC4G$4.VCCIO2, IC4G$8.VCCIO6, IC4G$9.VCCIO7, IC5.HOLD, IC5.VCC, IC5.WP, R11.2, R3.2, R4.2, X1.EN, X1.VCC
- net 1.8V_DCDC_SW: now also IC4.SW; no longer IC2.SW
- net DONE: now also IC1G$2.DONE, R9.1; no longer IC4G$2.DONE, R10.1
- net DRAM_+1V8: now also C49.1, C50.1, C51.1, FB8.1, IC9.VCC, IC9.VCCQ, R20.2; no longer C33.1, C34.1, C35.1, FB7.1, IC8.VCC, IC8.VCCQ
- net DRAM_CKN: now also IC1G$4.IO_L2N_T0_AD8N_15, IC9.!CK; no longer IC4G$6.PB28A, IC8.!CK
- net DRAM_CKP: now also IC1G$4.IO_L2P_T0_AD8P_15, IC9.CK; no longer IC4G$6.PB28B, IC8.CK
- net DRAM_CS: now also IC1G$4.IO_L1P_T0_AD0P_15, IC9.!CS; no longer IC4G$6.PB26A, IC8.!CS
- net DRAM_DQ0: now also IC1G$4.IO_L3N_T0_DQS_AD1N_15, IC9.DQ0; no longer IC4G$6.PB22A, IC8.DQ0
- net DRAM_DQ1: now also IC1G$4.IO_L4N_T0_15, IC9.DQ1; no longer IC4G$6.PB30B, IC8.DQ1
- net DRAM_DQ2: now also IC1G$4.IO_L7P_T1_AD2P_15, IC9.DQ2; no longer IC4G$6.PB18B, IC8.DQ2
- net DRAM_DQ3: now also IC1G$4.IO_L12N_T1_MRCC_15, IC9.DQ3; no longer IC4G$6.PB18A, IC8.DQ3
- net DRAM_DQ4: now also IC1G$4.IO_L7N_T1_AD2N_15, IC9.DQ4; no longer IC4G$6.PB16B, IC8.DQ4
- net DRAM_DQ5: now also IC1G$4.IO_L11N_T1_SRCC_15, IC9.DQ5; no longer IC4G$6.PB22B, IC8.DQ5
- net DRAM_DQ6: now also IC1G$4.IO_L5N_T0_AD9N_15, IC9.DQ6; no longer IC4G$6.PB24B, IC8.DQ6
- net DRAM_DQ7: now also IC1G$4.IO_L5P_T0_AD9P_15, IC9.DQ7; no longer IC4G$6.PB24A, IC8.DQ7
- net DRAM_NRST: now also IC9.!RESET, R20.1; no longer IC4G$6.PB20B, IC8.!RESET
- net DRAM_RWDS: now also IC1G$4.IO_L4P_T0_15, IC9.RWDS; no longer IC4G$6.PB30A, IC8.RWDS
- net FLASH_CS: now also IC1G$3.IO_L6P_T0_FCS_B_14, IC6.CS, R10.1; no longer IC4G$2.MCSN, IC5.CS, R11.1
- net FLASH_MISO: now also IC1G$3.IO_L1N_T0_D01_DIN_14, IC6.DO; no longer IC4G$2.MISO, IC5.DO
- net FLASH_MOSI: now also IC1G$3.IO_L1P_T0_D00_MOSI_14, IC6.DI; no longer IC4G$2.MOSI, IC5.DI
- net FLASH_SCK: now also IC1G$2.CCLK, IC6.CLK; no longer IC4G$2.MCLK, IC5.CLK
- net FT_+1V8: now also C46.1, C47.1, C48.1, FB7.2, IC8.VCORE1, IC8.VCORE2; no longer C30.1, C31.1, C32.1, FB6.2, IC7.VCORE1, IC7.VCORE2
- net FT_+3V3: now also C40.1, C41.1, C42.1, C43.1, FB6.2, IC7.VCC, IC8.VCCIO1, IC8.VCCIO2, IC8.VCCIO3, IC8.VPHY, IC8.VPLL, R11.1, R14.1; no longer C24.1, C25.1, C26.1, C27.1, FB5.2, IC6.VCC, IC7.VCCIO1, IC7.VCCIO2, IC7.VCCIO3, IC7.VPHY, IC7.VPLL, R12.1, R15.1
- net FT_CLK: now also IC1G$3.IO_L13P_T2_MRCC_14, IC8.ACBUS5; no longer IC4G$9.PL10A, IC7.ACBUS5
- net FT_D0: now also IC1G$3.IO_L10N_T1_D15_14, IC8.ADBUS0; no longer IC4G$9.PL17B, IC7.ADBUS0
- net FT_D1: now also IC1G$3.IO_L10P_T1_D14_14, IC8.ADBUS1; no longer IC4G$9.PL11A, IC7.ADBUS1
- net FT_D2: now also IC1G$3.IO_L16P_T2_CSI_B_14, IC8.ADBUS2; no longer IC4G$9.PL11B, IC7.ADBUS2
- net FT_D3: now also IC1G$3.IO_L16N_T2_A15_D31_14, IC8.ADBUS3; no longer IC4G$9.PL17A, IC7.ADBUS3
- net FT_D4: now also IC1G$3.IO_L15P_T2_DQS_RDWR_B_14, IC8.ADBUS4; no longer IC4G$9.PL3B, IC7.ADBUS4
- net FT_D5: now also IC1G$3.IO_L15N_T2_DQS_DOUT_CSO_B_14, IC8.ADBUS5; no longer IC4G$9.PL8B, IC7.ADBUS5
- net FT_D6: now also IC1G$3.IO_L17N_T2_A13_D29_14, IC8.ADBUS6; no longer IC4G$9.PL3A, IC7.ADBUS6
- net FT_D7: now also IC1G$3.IO_L17P_T2_A14_D30_14, IC8.ADBUS7; no longer IC4G$9.PL8A, IC7.ADBUS7
- net FT_NOE: now also IC1G$3.IO_L21P_T3_DQS_14, IC8.ACBUS6; no longer IC4G$9.PL10B, IC7.ACBUS6
- net FT_NRD: now also IC1G$3.IO_L20P_T3_A08_D24_14, IC8.ACBUS2; no longer IC4G$9.PL4A, IC7.ACBUS2
- net FT_NWR: now also IC1G$3.IO_L21N_T3_DQS_A06_D22_14, IC8.ACBUS3; no longer IC4G$9.PL6B, IC7.ACBUS3
- net FT_RXNF: now also IC1G$3.IO_L22N_T3_A04_D20_14, IC8.ACBUS0; no longer IC4G$9.PL4B, IC7.ACBUS0
- net FT_SIWU: now also IC1G$3.IO_L20N_T3_A07_D23_14, IC8.ACBUS4; no longer IC4G$9.PL19A, IC7.ACBUS4
- net FT_TXNE: now also IC1G$3.IO_L22P_T3_A05_D21_14, IC8.ACBUS1; no longer IC4G$9.PL6A, IC7.ACBUS1
- net GND: now also C36.2, C37.2, C38.2, C39.2, C40.2, C41.2, C42.2, C43.2, C44.2, C45.2, C46.2, C47.2, C48.2, C49.2, C50.2, C51.2, CON1.39, CON1.40, CON2.23, CON2.24, IC1G$1.GND, IC1G$1.GNDADC, IC1G$1.VCCBAT, IC1G$2.DXN, IC1G$2.DXP, IC1G$2.M1, IC1G$2.M2, IC1G$2.VN, IC1G$2.VP, IC1G$2.VREFN, IC1G$2.VREFP, IC4.GND, IC6.GND, IC7.VSS, IC8.GND1, IC8.GND2, IC8.GND3, IC8.HT, IC8.TEST, IC9.VSS, IC9.VSSQ, R13.2, R15.1, R4.1, TP5.1; no longer CON1.31, CON1.32, CON1.52, CON2.14, CON2.15, CON2.16, CON2.33, CON2.34, CON2.35, CON2.36, CON2.37, CON2.38, CON2.39, CON2.40, IC1.GND, IC4G$1.GND, IC4G$10.VSSADC, IC6.VSS, IC7.GND1, IC7.GND2, IC7.GND3, IC7.HT, IC7.TEST, IC8.VSS, IC8.VSSQ, R14.2, R5.1, X2.GND
- net JTAG_TCK: now also IC1G$2.TCK, IC8.BDBUS0, TP3.1; no longer IC4G$3.TCK, IC7.BDBUS0, R5.2
- net JTAG_TDI: now also IC1G$2.TDI, IC8.BDBUS1, R5.1, TP2.1; no longer IC4G$3.TDI, IC7.BDBUS1, R4.1
- net JTAG_TDO: now also IC1G$2.TDO, IC8.BDBUS2, TP4.1; no longer IC4G$3.TDO, IC7.BDBUS2, R3.1
- net JTAG_TMS: now also IC1G$2.TMS, IC8.BDBUS3, TP1.1; no longer IC4G$3.TMS, IC7.BDBUS3
- net LED0: now also IC1G$3.IO_L24N_T3_A00_D16_14; no longer IC4G$3.PR20A
- net LED1: now also IC1G$3.IO_L24P_T3_A01_D17_14; no longer IC4G$3.PR20B
- net LED2: now also IC1G$3.IO_L23N_T3_A02_D18_14; no longer IC4G$3.PR19A
- net N$1: now also D6.K; no longer D5.K
- net N$10: now also IC7.DI, IC8.EEDATA, R12.2; no longer IC6.DI, IC7.EEDATA, R13.2
- net N$11: now also IC7.CS, IC8.EECS; no longer IC6.CS, IC7.EECS
- net N$12: now also IC7.DO, R11.2, R12.1; no longer IC6.DO, R12.2, R13.1
- net N$13: now also C45.1, IC8.OSCO, X1.2; no longer C29.1, IC7.OSCO, X2.2
- net N$14: now also C44.1, IC8.OSCI, X1.1; no longer C28.1, IC7.OSCI, X2.1
- net N$15: now also IC8.REF, R13.1; no longer IC7.REF, R14.1
- net N$16: now also IC8.RESET#, R14.2; no longer IC7.RESET#, R15.2
- net N$2: now also R15.2; no longer R16.2
- net N$3: now also R16.2; no longer R17.2
- net N$4: now also R17.2; no longer R18.2
- net N$9: now also IC7.CLK, IC8.EECLK; no longer IC6.CLK, IC7.EECLK
- net USB_DM: now also IC8.DM; no longer IC7.DM
- net USB_DP: now also IC8.DP; no longer IC7.DP
- net VIN_DCDC: now also C6.1, IC2.IN, IC3.EN, IC3.IN, IC4.EN, IC4.VIN, IC5.EN, IC5.VIN; no longer IC1.EN, IC1.IN, IC2.VIN
Other:
- note removed: "HV"
- note removed: "LV"
- moved on the sheet: C1, C10, C11, C12, C13, C14, C15, C16, C17, C18, C19, C2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

Commit message: via打てば終わり
Parts:
- D2: value LED0 -> 0
- D3: value LED1 -> 1
- D4: value LED2 -> 2
- D5: value LED2 -> 3
- D6: value PWR -> P
- IC8: value FT2232H-2 -> FT2232H
Connections:
- net +1V8: no longer CON1.55, CON1.56
- net +2V5: now also CON1.55, CON1.56; no longer CON2.49, CON2.50
- net +3V3: now also CON2.49, CON2.50
Other:
- note added: "DC-DC / LDO"
- moved on the sheet: C1, C16, C17, C18, C19, C2, C20, C21, C22, C23, C3, C39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

Commit message: 発注
Parts:
- added C52, C53, C54: 10u, my_rcl:C-2012
- C11, C12: value 1u -> 0.1u; device my_rcl:C-1005 -> my_rcl:C-1608
- C16, C4: value 10u -> 1u; device my_rcl:C-1608 -> my_rcl:C-1005
- C20: device my_rcl:C-2012 -> my_rcl:C-1608
- C26: value 1u -> 10u; device my_rcl:C-1005 -> my_rcl:C-2012
- C39, C5: value 0.1u -> 1u; device my_rcl:C-1608 -> my_rcl:C-1005
- C40: value 10u -> 0.1u
- C41, C47, C6: value 0.1u -> 10u
- C44: value 22p -> 0.1u
- C46: value 10u -> 22p
- C50: value 10u -> 0.1u; device my_rcl:C-2012 -> my_rcl:C-1608
- R11: value 10k -> 1k
- R13: value 12.1k -> 10k
- R17: value 1k -> 12.1k
Connections:
- net +1V0: now also C16.1, C26.1, C4.1, C53.1; no longer C11.1, C23.1
- net +1V0_DCDC: now also C20.1; no longer C19.1
- net +1V8: now also C25.1, C32.1, C34.1, C36.1, C5.1, C54.1; no longer C12.1, C22.1, C31.1, C33.1, C35.1
- net +1V8_DCDC: now also C19.1; no longer C18.1
- net +2V5: now also C22.1; no longer C21.1
- net +2V5_LDO: now also C18.1; no longer C17.1
- net +3V3: now also C21.1, C33.1, C35.1, C40.1; no longer C20.1, C32.1, C34.1, C36.1
- net +3V3_LDO: now also C17.1; no longer C16.1
- net DRAM_+1V8: now also C52.1; no longer C49.1
- net FT_+1V8: now also C49.1; no longer C46.1
- net FT_+3V3: now also C44.1, R13.1, R18.1; no longer C40.1, R11.1, R14.1
- net GND: now also C52.2, C53.2, C54.2, R11.1, R12.1, R14.1, R17.2; no longer R13.2, R16.1, R17.1, R18.1
- net N$10: now also R16.2; no longer R12.2
- net N$12: now also R13.2, R16.1; no longer R11.2, R12.1
- net N$13: now also C46.1; no longer C45.1
- net N$14: now also C45.1; no longer C44.1
- net N$15: now also R17.1; no longer R13.1
- net N$16: now also R18.2; no longer R14.2
- net N$2: now also R11.2; no longer R15.2
- net N$3: now also R12.2; no longer R16.2
- net N$4: now also R14.2; no longer R17.2
- net N$5: now also R15.2; no longer R18.2
- net VCCO34: now also C23.1, C27.1, C29.1; no longer C24.1, C26.1, C28.1
- net VCCO35: now also C24.1, C28.1, C31.1; no longer C25.1, C27.1, C29.1
- net VIN_DCDC: now also C11.1, C12.1; no longer C4.1, C5.1
Other:
- moved on the sheet: C10, C11, C12, C16, C17, C18, C19, C20, C21, C22, C23, C24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

Commit message: OSCを追加して再発注
Parts:
- added C55, C56: 0.1u, my_rcl:C-1608
- added C57: 10u, my_rcl:C-2012
- added J3: 25M, my_rcl:SJ-1608
- added R21: 1k, my_rcl:R-1608
- added X2: 12MHz, my_rcl:CRYSTAL2
- C10, C9: value 1u -> 0.1u; device my_rcl:C-1005 -> my_rcl:C-1608
- C11, C12, C40, C42, C43: value 0.1u -> 1u; device my_rcl:C-1608 -> my_rcl:C-1005
- C27, C28: value 1u -> 10u; device my_rcl:C-1005 -> my_rcl:C-2012
- C29, C30: value 1u -> 10u; device my_rcl:C-1005 -> my_rcl:C-3216
- C4: value 1u -> 10u; device my_rcl:C-1005 -> my_rcl:C-1608
- C41, C6: value 10u -> 1u; device my_rcl:C-1608 -> my_rcl:C-1005
- C45: value 22p -> 0.1u
- C46: value 22p -> 10u
- C47: value 10u -> 0.1u
- C50, C51: value 0.1u -> 22p
- C52: device my_rcl:C-2012 -> my_rcl:C-1608
- C53, C54: value 10u -> 0.1u; device my_rcl:C-2012 -> my_rcl:C-1608
- R11, R14: value 1k -> 10k
- R13: value 10k -> 1k
- R17: value 12.1k -> 1k
- R18: value 1k -> 12.1k
- X1: value 12MHz -> 25MHz; device my_rcl:CRYSTAL2 -> my_rcl:OSC-KC3225
Connections:
- new net CLK_25M: IC1G$3.IO_L13P_T2_MRCC_14, J3.2
- new net N$8: J3.1, X1.OUT
- net +1V0: now also C11.1, C24.1, C30.1, C5.1; no longer C4.1, C53.1, C9.1
- net +1V8: now also C12.1, C23.1, C29.1, C38.1, C40.1, C6.1; no longer C10.1, C32.1, C34.1, C5.1, C54.1
- net +3V3: now also C41.1, C42.1, C43.1, C44.1, C45.1, R11.2, X1.EN, X1.VCC; no longer C33.1, C35.1, C38.1, C40.1, R6.2
- net DONE: now also R10.1; no longer R9.1
- net DRAM_+1V8: now also C55.1, C56.1, C57.1, R21.2; no longer C50.1, C51.1, C52.1, R20.2
- net DRAM_NRST: now also R21.1; no longer R20.1
- net FLASH_CS: now also R11.1; no longer R10.1
- net FT_+1V8: now also C52.1, C53.1, C54.1; no longer C47.1, C48.1, C49.1
- net FT_+3V3: now also C46.1, C47.1, C48.1, C49.1, R14.1, R19.1; no longer C41.1, C42.1, C43.1, C44.1, R13.1, R18.1
- net FT_CLK: now also IC1G$3.IO_L14P_T2_SRCC_14; no longer IC1G$3.IO_L13P_T2_MRCC_14
- net GND: now also C55.2, C56.2, C57.2, R13.1, R16.1, R18.2, R20.1, R6.1, X2.GND; no longer R11.1, R14.1, R17.2, R19.1
- net INIT_B: now also R8.1; no longer R7.1
- net JTAG_TCK: now also R6.2
- net JTAG_TMS: now also R7.1; no longer R6.1
- net N$1: now also R20.2; no longer R19.2
- net N$10: now also R17.2; no longer R16.2
- net N$12: now also R14.2, R17.1; no longer R13.2, R16.1
- net N$13: now also C51.1, X2.2; no longer C46.1, X1.2
- net N$14: now also C50.1, X2.1; no longer C45.1, X1.1
- net N$15: now also R18.1; no longer R17.1
- net N$16: now also R19.2; no longer R18.2
- net N$2: now also R12.2; no longer R11.2
- net N$3: now also R13.2; no longer R12.2
- net N$4: now also R15.2; no longer R14.2
- net N$5: now also R16.2; no longer R15.2
- net PROGRAM_B: now also R9.1; no longer R8.1
- net VCCO34: now also C31.1, C33.1; no longer C23.1, C29.1
- net VCCO35: now also C32.1, C34.1, C35.1; no longer C24.1, C30.1, C31.1
- net VIN_DCDC: now also C10.1, C4.1, C9.1; no longer C11.1, C12.1, C6.1
Other:
- moved on the sheet: C1, C10, C11, C12, C17, C18, C19, C2, C20, C21, C22, C23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

Commit message: Type-C
Parts:
- removed C30: 10u, my_rcl:C-3216
- added R22, R23: 5.1k, my_rcl:R-1608
- CON3: value USB-SC -> USB-C; device my_connector:USB-SC -> my_connector:USB-C
- J1, J2: device my_rcl:SJ-3 -> my_rcl:SJ-3-1608
- TP1, TP2, TP3, TP4, TP5: device my_connector:TESTPIN-PAD -> my_connector:TESTPIN-PAD-SMALL
Connections:
- new net N$6: CON3.CC1, R22.2
- new net N$7: CON3.CC2, R23.2
- net +1V0: no longer C30.1
- net GND: now also R22.1, R23.1; no longer C30.2

Commit message: 微修正
Parts:
- removed D1: USB, my_rcl:SBD-1A2
- added FB9: USB, my_rcl:FB
Connections:
- net USB_+5V: now also FB9.1; no longer D1.A
- net VIN: now also FB9.2; no longer D1.K

Commit message: 発注
Parts:
- added C30, C58: 0.1u, my_rcl:C-1608
- IC4: value MPM3804 -> MPM3811
Connections:
- net +1V8: now also C30.1, C58.1, CON2.13, CON2.14, CON2.15, CON2.16; no longer CON2.45, CON2.46, CON2.47, CON2.48
- net +3V3: now also CON2.10, CON2.11, CON2.12, CON2.9; no longer CON2.49, CON2.50, CON2.51, CON2.52
- net GND: now also C30.2, C58.2, CON2.17, CON2.18, CON2.19, CON2.20, CON2.37, CON2.38, CON2.5, CON2.59, CON2.6, CON2.60, CON2.7, CON2.8; no longer CON2.1, CON2.2, CON2.23, CON2.24, CON2.41, CON2.42, CON2.43, CON2.44, CON2.53, CON2.54, CON2.55, CON2.56
- net IO0_14: now also CON2.35; no longer CON2.26
- net IO10N_15: now also CON2.54; no longer CON2.7
- net IO10P_15: now also CON2.52; no longer CON2.9
- net IO11N_14: now also CON2.21; no longer CON2.40
- net IO11P_14: now also CON2.23; no longer CON2.38
- net IO12N_14: now also CON2.29; no longer CON2.32
- net IO12P_14: now also CON2.31; no longer CON2.30
- net IO13N_15: now also CON2.49; no longer CON2.12
- net IO13P_15: now also CON2.47; no longer CON2.14
- net IO15N_15: now also CON2.51; no longer CON2.10
- net IO15P_15: now also CON2.53; no longer CON2.8
- net IO17N_15: now also CON2.50; no longer CON2.11
- net IO17P_15: now also CON2.48; no longer CON2.13
- net IO21N_15: now also CON2.45; no longer CON2.16
- net IO21P_15: now also CON2.43; no longer CON2.18
- net IO22N_15: now also CON2.46; no longer CON2.15
- net IO22P_15: now also CON2.44; no longer CON2.17
- net IO23N_15: now also CON2.40; no longer CON2.21
- net IO23P_15: now also CON2.42; no longer CON2.19
- net IO24N_15: now also CON2.41; no longer CON2.20
- net IO24P_15: now also CON2.39; no longer CON2.22
- net IO2N_14: now also CON2.34; no longer CON2.27
- net IO2P_14: now also CON2.36; no longer CON2.25
- net IO4N_14: now also CON2.30; no longer CON2.31
- net IO4P_14: now also CON2.32; no longer CON2.29
- net IO5P_14: now also CON2.33; no longer CON2.28
- net IO7N_14: now also CON2.26; no longer CON2.35
- net IO7P_14: now also CON2.28; no longer CON2.33
- net IO8N_14: now also CON2.22; no longer CON2.39
- net IO8N_15: now also CON2.57; no longer CON2.4
- net IO8P_14: now also CON2.24; no longer CON2.37
- net IO8P_15: now also CON2.55; no longer CON2.6
- net IO9N_14: now also CON2.25; no longer CON2.36
- net IO9N_15: now also CON2.58; no longer CON2.3
- net IO9P_14: now also CON2.27; no longer CON2.34
- net IO9P_15: now also CON2.56; no longer CON2.5
- net VIN: now also CON2.1, CON2.2, CON2.3, CON2.4; no longer CON2.57, CON2.58, CON2.59, CON2.60
Other:
- moved on the sheet: C1, C10, C17, C18, C19, C2, C20, C21, C22, C23, C24, C25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

Commit message: 微修正
Parts:
- removed D6: P, my_rcl:LED-SMD1608
- added C59, C60: 1u, my_rcl:C-1608
- added C61: 10u, my_rcl:C-2012
- added D1: 0, my_rcl:LED-SMD1608
- C10, C44, C45, C47: value 0.1u -> 1u; device my_rcl:C-1608 -> my_rcl:C-1005
- C11, C7, C8: value 1u -> 4.7u; device my_rcl:C-1005 -> my_rcl:C-1608
- C17, C18, C46: value 10u -> 1u; device my_rcl:C-1608 -> my_rcl:C-1005
- C21, C22: value 10u -> 1u; device my_rcl:C-2012 -> my_rcl:C-1005
- C23, C24: device my_rcl:C-2012 -> my_rcl:C-1608
- C29: device my_rcl:C-3216 -> my_rcl:C-2012
- C30: value 0.1u -> 10u; device my_rcl:C-1608 -> my_rcl:C-2012
- C31: value 1u -> 10u; device my_rcl:C-1005 -> my_rcl:C-3216
- C32, C33: value 1u -> 10u; device my_rcl:C-1005 -> my_rcl:C-2012
- C34, C5, C6: value 1u -> 0.1u; device my_rcl:C-1005 -> my_rcl:C-1608
- C50: value 22p -> 10u
- C51: value 22p -> 0.1u
- C52: value 10u -> 0.1u
- C54, C55: value 0.1u -> 22p
- C56: value 0.1u -> 10u
- C57: value 10u -> 0.1u; device my_rcl:C-2012 -> my_rcl:C-1608
- C9: value 0.1u -> 4.7u
- D2: value 0 -> 1
- D3: value 1 -> 2
- D4: value 2 -> 3
- D5: value 3 -> P
- FB1: value VIN -> USB
- FB2: value 3.3V -> VIN
- FB3: value 2.5V -> 3.3V
- FB4: value 1.8V -> 2.5V
- FB5: value 1.0V -> 1.8V
- FB6: value FT -> 1.0V
- FB8: value DRAM -> FT
- FB9: value USB -> DRAM
- R16, R17: value 1k -> 5.1k
- R18: value 12.1k -> 1k
- R20: value 1k -> 12.1k
- R22, R23: value 5.1k -> 1k
- X1: value 25MHz -> OSC
Connections:
- net +1V0: now also C10.1, C12.1, C14.1, C18.1, C22.1, C28.1, C30.1, C8.1, FB6.2; no longer C11.1, C13.1, C15.1, C24.1, C26.1, C5.1, C7.1, FB5.2
- net +1V0_DCDC: now also C24.1, FB6.1; no longer C20.1, FB5.1
- net +1V8: now also C11.1, C13.1, C15.1, C17.1, C21.1, C27.1, C31.1, C34.1, C42.1, C44.1, C7.1, C9.1, FB5.2, FB8.1, FB9.2; no longer C12.1, C14.1, C23.1, C25.1, C30.1, C36.1, C38.1, C58.1, C6.1, C8.1, FB4.2, FB7.1, FB8.2
- net +1V8_DCDC: now also C23.1, FB5.1; no longer C19.1, FB4.1
- net +2V5: now also C26.1, FB4.2; no longer C22.1, FB3.2
- net +2V5_LDO: now also C20.1, FB4.1; no longer C18.1, FB3.1
- net +3V3: now also C25.1, C46.1, C47.1, C48.1, C49.1, D5.A, FB3.2, FB7.1; no longer C21.1, C37.1, C39.1, C42.1, C44.1, D6.A, FB2.2, FB6.1
- net +3V3_LDO: now also C19.1, FB3.1; no longer C17.1, FB2.1
- net DRAM_+1V8: now also C59.1, C60.1, C61.1, FB9.1, R23.2; no longer C55.1, C56.1, C57.1, FB8.1, R21.2
- net DRAM_NRST: now also R23.1; no longer R21.1
- net FT_+1V8: now also C56.1, C57.1, C58.1, FB8.2; no longer C52.1, C53.1, C54.1, FB7.2
- net FT_+3V3: now also C50.1, C51.1, C52.1, C53.1, FB7.2, R21.1; no longer C46.1, C47.1, C48.1, C49.1, FB6.2, R19.1
- net GND: now also C59.2, C60.2, C61.2, R17.1, R18.1, R20.2; no longer R18.2, R20.1, R23.1
- net LED0: now also D1.A; no longer D2.A
- net LED1: now also D2.A; no longer D3.A
- net LED2: now also D3.A; no longer D4.A
- net LED3: now also D4.A; no longer D5.A
- net N$1: now also D5.K, R22.2; no longer D6.K, R20.2
- net N$10: now also R19.2; no longer R17.2
- net N$12: now also R19.1; no longer R17.1
- net N$13: now also C55.1; no longer C51.1
- net N$14: now also C54.1; no longer C50.1
- net N$15: now also R20.1; no longer R18.1
- net N$16: now also R21.2; no longer R19.2
- net N$2: now also D1.K; no longer D2.K
- net N$3: now also D2.K; no longer D3.K
- net N$4: now also D3.K; no longer D4.K
- net N$5: now also D4.K, R18.2; no longer D5.K, R16.2
- net N$6: now also R16.2; no longer R22.2
- net N$7: now also R17.2; no longer R23.2
- net USB_+5V: now also FB1.1; no longer FB9.1
- net VCCO34: now also C32.1, C35.1, C37.1; no longer C27.1, C31.1, C33.1
- net VCCO35: now also C33.1, C36.1, C38.1, C39.1; no longer C28.1, C32.1, C34.1, C35.1
- net VIN: now also FB1.2, FB2.1; no longer FB1.1, FB9.2
- net VIN_DCDC: now also C5.1, C6.1, FB2.2; no longer C10.1, C9.1, FB1.2
Other:
- moved on the sheet: C10, C11, C12, C13, C14, C15, C16, C17, C18, C19, C20, C21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
