File: ADC3_FPGA_BGA.sch (EAGLE design)
At the start: 120 parts, among them CON1 MEZZANINE_2X30, CON2 MEZZANINE_2X30, CON3 USB-C, IC1 ARTIX7-FTG256, IC2 3.3V, IC3 2.5V, IC4 MPM3811, IC5 MPM3804, IC6 EEPROM, IC7 93LC56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

Commit message: Create README.md
Connections:
- net DRAM_NRST: now also IC1G$4.IO_L6P_T0_15
- net FT_+1V8: now also IC8.VCORE@1, IC8.VCORE@2; no longer IC8.VCORE1, IC8.VCORE2
- net FT_+3V3: now also IC8.VCCIO@1, IC8.VCCIO@2, IC8.VCCIO@3; no longer IC8.VCCIO1, IC8.VCCIO2, IC8.VCCIO3
- net GND: now also IC8.GND@1, IC8.GND@2, IC8.GND@3; no longer IC8.GND1, IC8.GND2, IC8.GND3
Other:
- note added: "FPGA"
- note added: "I/O Connector"
- note removed: "FPGA IO"
- moved on the sheet: C1, C10, C11, C12, C13, C14, C15, C16, C17, C18, C19, C2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
